File: Hermes/hermes_v1/hermes_v1.kicad_pcb (KiCad board)
At the start: 2 copper layers, 65 x 30 mm, 62 parts, among them IC1 LD39200PU33R, J1 Raspberry Pi Zero, J2 FCC_BOOT, J3 FCC_RESET, J6 2.54mm, J7 Conn_02x06_Odd_Even, J8 Connector_USB_B_Micro, P1 5V_BAT, P2 GND_BAT, U1 RP2040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

Commit message: old
Routing:
- net FC_USB_D+: track 0.00 -> 5.58 mm
- net FC_USB_D-: track 0.00 -> 5.20 mm
Other:
- net class usb added: clearance 0.13, trace_width 0.8, via_dia 0.8, via_drill 0.4
Changed lines of the file:
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@@
     (thickness 1.6)
     (drawings 10)
-    (tracks 457)
+    (tracks 467)
     (zones 0)
     (modules 62)
@@
     (user_trace_width 0.4)
     (user_trace_width 0.45)
-    (user_trace_width 0.5)
+    (user_trace_width 0.6)
+    (user_trace_width 0.8)
     (user_trace_width 1.5)
     (trace_clearance 0.2)
@@
     (add_net VCC)
   )
+  (net_class usb ""
+    (clearance 0.13)
+    (trace_width 0.8)
+    (via_dia 0.8)
+    (via_drill 0.4)
+    (uvia_dia 0.3)
+    (uvia_drill 0.1)
+    (diff_pair_width 0.8)
+    (diff_pair_gap 0.13)
+  )
+  (module Resistor_SMD:R_0402_1005Metric_Pad0.72x0.64mm_HandSolder (layer F.Cu)
+    (at 125.2855 66.294)
+    (descr "Resistor SMD 0402 (1005 Metric), square (rectangular) end terminal, IPC_7351 nominal with elongated pad for handsoldering. (Body size source: IPC-SM-782 page 72, https://www.pcb-3d.com/wordpress/wp-content/uploads/ipc-sm-782a_amendment_1_and_2.pdf), generated with kicad-footprint-generator")
+    (tags "resistor handsolder")
+    (attr smd)
+    (fp_text reference R10 (at -2.286 0) (layer F.SilkS)
+      (effects (font (size 0.7 0.7) (thickness 0.15)))
+    )
+    (fp_text value 27 (at -21.971 -2.54 -90) (layer F.Fab)
+      (effects (font (size 1 1) (thickness 0.15)))
+    )
+    (fp_line (start 1.1 0.47) (end -1.1 0.47) (layer F.CrtYd) (width 0.05))
+    (fp_line (start 1.1 -0.47) (end 1.1 0.47) (layer F.CrtYd) (width 0.05))
+    (fp_line (start -1.1 -0.47) (end 1.1 -0.47) (layer F.CrtYd) (width 0.05))
+    (fp_line (start -1.1 0.47) (end -1.1 -0.47) (layer F.CrtYd) (width 0.05))
+    (fp_line (start -0.167621 0.38) (end 0.167621 0.38) (layer F.SilkS) (width 0.12))
+    (fp_line (start -0.167621 -0.38) (end 0.167621 -0.38) (layer F.SilkS) (width 0.12))
+    (fp_line (start 0.525 0.27) (end -0.525 0.27) (layer F.Fab) (width 0.1))
+    (fp_line (start 0.525 -0.27) (end 0.525 0.27) (layer F.Fab) (width 0.1))
+    (fp_line (start -0.525 -0.27) (end 0.525 -0.27) (layer F.Fab) (width 0.1))
+    (fp_line (start -0.525 0.27) (end -0.525 -0.27) (layer F.Fab) (width 0.1))
+    (fp_text user %R (at 0 0) (layer F.Fab)
+      (effects (font (size 0.26 0.26) (thickness 0.04)))
+    )
+    (pad 2 smd roundrect (at 0.5975 0) (size 0.715 0.64) (layers F.Cu F.Paste F.Mask) (roundrect_rratio 0.25)
+      (net 35 "Net-(R10-Pad2)"))
+    (pad 1 smd roundrect (at -0.5975 0) (size 0.715 0.64) (layers F.Cu F.Paste F.Mask) (roundrect_rratio 0.25)
+      (net 34 FC_USB_D-))
+    (model ${KICAD6_3DMODEL_DIR}/Resistor_SMD.3dshapes/R_0402_1005Metric.wrl
+      (at (xyz 0 0 0))
+      (scale (xyz 1 1 1))
+      (rotate (xyz 0 0 0))
+    )
+  )
   (module RP2040:QFN40P695X695X90-57T320N (layer F.Cu)
     (at 132.0165 68.072 90)
@@
   )
   (module Resistor_SMD:R_0402_1005Metric_Pad0.72x0.64mm_HandSolder (layer F.Cu)
-    (at 125.2855 66.294)
-    (descr "Resistor SMD 0402 (1005 Metric), square (rectangular) end terminal, IPC_7351 nominal with elongated pad for handsoldering. (Body size source: IPC-SM-782 page 72, https://www.pcb-3d.com/wordpress/wp-content/uploads/ipc-sm-782a_amendment_1_and_2.pdf), generated with kicad-footprint-generator")
-    (tags "resistor handsolder")
-    (attr smd)
-    (fp_text reference R10 (at -2.286 0) (layer F.SilkS)
-      (effects (font (size 0.7 0.7) (thickness 0.15)))
-    )
-    (fp_text value 27 (at -21.971 -2.54 -90) (layer F.Fab)
-      (effects (font (size 1 1) (thickness 0.15)))
-    )
-    (fp_line (start 1.1 0.47) (end -1.1 0.47) (layer F.CrtYd) (width 0.05))
-    (fp_line (start 1.1 -0.47) (end 1.1 0.47) (layer F.CrtYd) (width 0.05))
-    (fp_line (start -1.1 -0.47) (end 1.1 -0.47) (layer F.CrtYd) (width 0.05))
-    (fp_line (start -1.1 0.47) (end -1.1 -0.47) (layer F.CrtYd) (width 0.05))
-    (fp_line (start -0.167621 0.38) (end 0.167621 0.38) (layer F.SilkS) (width 0.12))
-    (fp_line (start -0.167621 -0.38) (end 0.167621 -0.38) (layer F.SilkS) (width 0.12))
-    (fp_line (start 0.525 0.27) (end -0.525 0.27) (layer F.Fab) (width 0.1))
-    (fp_line (start 0.525 -0.27) (end 0.525 0.27) (layer F.Fab) (width 0.1))
-    (fp_line (start -0.525 -0.27) (end 0.525 -0.27) (layer F.Fab) (width 0.1))
-    (fp_line (start -0.525 0.27) (end -0.525 -0.27) (layer F.Fab) (width 0.1))
-    (fp_text user %R (at 0 0) (layer F.Fab)
-      (effects (font (size 0.26 0.26) (thickness 0.04)))
-    )
-    (pad 2 smd roundrect (at 0.5975 0) (size 0.715 0.64) (layers F.Cu F.Paste F.Mask) (roundrect_rratio 0.25)
-      (net 35 "Net-(R10-Pad2)"))
-    (pad 1 smd roundrect (at -0.5975 0) (size 0.715 0.64) (layers F.Cu F.Paste F.Mask) (roundrect_rratio 0.25)
-      (net 34 FC_USB_D-))
-    (model ${KICAD6_3DMODEL_DIR}/Resistor_SMD.3dshapes/R_0402_1005Metric.wrl
-      (at (xyz 0 0 0))
-      (scale (xyz 1 1 1))
-      (rotate (xyz 0 0 0))
-    )
-  )
-  (module Resistor_SMD:R_0402_1005Metric_Pad0.72x0.64mm_HandSolder (layer F.Cu)
     (at 125.2855 67.437)
     (descr "Resistor SMD 0402 (1005 Metric), square (rectangular) end terminal, IPC_7351 nominal with elongated pad for handsoldering. (Body size source: IPC-SM-782 page 72, https://www.pcb-3d.com/wordpress/wp-content/uploads/ipc-sm-782a_amendment_1_and_2.pdf), generated with kicad-footprint-generator")
@@
   (segment (start 127.219905 67.072) (end 127.209904 67.061999) (width 0.2) (layer F.Cu) (net 32))
   (segment (start 128.609 67.072) (end 127.219905 67.072) (width 0.2) (layer F.Cu) (net 32))
+  (segment (start 123.995 66.744) (end 124.688 67.437) (width 0.2) (layer F.Cu) (net 33))
+  (segment (start 121.436502 66.744) (end 123.995 66.744) (width 0.2) (layer F.Cu) (net 33))
+  (segment (start 121.120501 67.060001) (end 121.436502 66.744) (width 0.2) (layer F.Cu) (net 33))
+  (segment (start 119.880499 67.060001) (end 121.120501 67.060001) (width 0.2) (layer F.Cu) (net 33))
+  (segment (start 119.6305 67.31) (end 119.880499 67.060001) (width 0.2) (layer F.Cu) (net 33))
+  (segment (start 119.6305 66.51) (end 119.680966 66.51) (width 0.4) (layer F.Cu) (net 34))
+  (segment (start 120.010103 66.294) (end 123.995 66.294) (width 0.2) (layer F.Cu) (net 34))
+  (segment (start 119.6305 66.51) (end 119.794103 66.51) (width 0.2) (layer F.Cu) (net 34))
+  (segment (start 123.995 66.294) (end 124.688 66.294) (width 0.2) (layer F.Cu) (net 34))
+  (segment (start 119.794103 66.51) (end 120.010103 66.294) (width 0.2) (layer F.Cu) (net 34))
   (segment (start 125.883 66.294) (end 126.002 66.294) (width 0.2) (layer F.Cu) (net 35))
   (segment (start 126.250989 66.661989) (end 125.883 66.294) (width 0.2) (layer F.Cu) (net 35))
