File: Hermes/hermes_v1/hermes_v1.kicad_pcb (KiCad board)
At the start: 4 copper layers, 32.7 x 49.9 mm, 77 parts, among them J2 Connector_USB_B_Micro, J3 Conn_01x07, J4 Conn_02x07_Odd_Even, J5 Additional IO, J6 Micro_SD_Card, J7 IO Power, P1 ESC1_VCC, P2 ESC1_GND, P3 LIPO_VCC, P4 LIPO_GND, P5 ESC2_VCC, P6 ESC2_GND, SW1 BOOT_SEL, SW2 RESET, U1 TPS5430DDAR, U2 LD1117S33TR_SOT223, U3 RP2040, U4 W25Q128JVS, U5 MPU-6050, U6 MPL3115A2, U7 USBLC6-2P6, Y1 12MHz ±30ppm 12pF 50Ω SMD-503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

Commit message: added piUAV & Proteus_v1
Parts:
- removed REF**: OSHW-Logo2_7.3x6mm_SilkScreen, Symbol:OSHW-Logo2_7.3x6mm_SilkScreen
- added H1: MountingHole, MountingHole:MountingHole_2.2mm_M2_DIN965_Pad, F.Cu at (225.2, 46.0)
- added H2: MountingHole, MountingHole:MountingHole_2.2mm_M2_DIN965_Pad, F.Cu at (188.1, 91.2)
- added H3: MountingHole, MountingHole:MountingHole_2.2mm_M2_DIN965_Pad, F.Cu at (225.2, 91.2)
- added H4: MountingHole, MountingHole:MountingHole_2.2mm_M2_DIN965_Pad, F.Cu at (188.1, 46.0)
- moved C21 0.08 mm to (215.4, 75.0)
Routing:
- added copper zone on In1.Cu, net GND
- removed copper zone on GND, net GND
Other:
- board size 32.7 x 49.9 mm -> 41.8 x 49.9 mm
- net class Default removed
- net class usb removed
- board text added: "HERMES"
- board text removed: "KÁRMÁN"

Commit message: Hermes v2
Parts:
- removed C21, C24: 0.1u, Capacitor_SMD:C_0402_1005Metric_Pad0.74x0.62mm_HandSolder
- removed C23: 10u, Capacitor_SMD:C_0402_1005Metric_Pad0.74x0.62mm_HandSolder
- removed H1, H2, H3, H4: MountingHole, MountingHole:MountingHole_2.2mm_M2_DIN965_Pad
- removed J4: Conn_02x07_Odd_Even, Connector_PinHeader_2.54mm:PinHeader_2x07_P2.54mm_Vertical
- removed J5: Additional IO, Connector_PinHeader_2.54mm:PinHeader_2x03_P2.54mm_Vertical
- removed J7: IO Power, Connector_PinHeader_2.54mm:PinHeader_2x03_P2.54mm_Vertical
- removed R10, R11: 4k7, Resistor_SMD:R_0402_1005Metric_Pad0.72x0.64mm_HandSolder
- removed R8: DNP, Resistor_SMD:R_0402_1005Metric_Pad0.72x0.64mm_HandSolder
- removed TP1: GND_BAT_Probe, TestPoint:TestPoint_Pad_D1.0mm
- removed TP2: 5V_BAT_Probe, TestPoint:TestPoint_Pad_D1.0mm
- removed U6: MPL3115A2, Package_LGA:NXP_LGA-8_3x5mm_P1.25mm_H1.1mm
- added ?: , RPi_Hat:RPi_Hat_Mounting_Hole, F.Cu at (243.0, 38.1)
- added ?: , RPi_Hat:RPi_Hat_Mounting_Hole, F.Cu at (266.0, 38.1)
- added ?: , RPi_Hat:RPi_Hat_Mounting_Hole, F.Cu at (243.0, 96.1)
- added ?: , RPi_Hat:RPi_Hat_Mounting_Hole, F.Cu at (266.0, 96.1)
- added J1: Conn_02x20_Odd_Even, Connector_PinSocket_2.54mm:PinSocket_2x20_P2.54mm_Vertical, F.Cu at (267.3, 43.0)
- added J8: Conn_01x08, Connector_PinHeader_2.54mm:PinHeader_1x08_P2.54mm_Vertical, F.Cu at (261.0, 86.2)
- added J9: Conn_02x08_Odd_Even, Connector_PinHeader_2.54mm:PinHeader_2x08_P2.54mm_Vertical, F.Cu at (243.2, 91.3)
- added kibuzzard-62AD2A8F: G***, kibuzzard-62AD2A8F, F.Cu at (244.7, 71.7)
- added kibuzzard-62ADC3D6: G***, kibuzzard-62ADC3D6, F.Cu at (240.7, 86.1)
- added kibuzzard-62ADC3E7: G***, kibuzzard-62ADC3E7, F.Cu at (240.6, 88.8)
- added kibuzzard-62ADC3FE: G***, kibuzzard-62ADC3FE, F.Cu at (240.7, 91.3)
- added kibuzzard-62ADC89D: G***, kibuzzard-62ADC89D, F.Cu at (251.8, 80.0)
- added kibuzzard-62ADCC2A: G***, kibuzzard-62ADCC2A, F.Cu at (255.8, 99.0)
- added kibuzzard-62ADCC37: G***, kibuzzard-62ADCC37, F.Cu at (253.3, 99.0)
- added kibuzzard-62ADCC62: G***, kibuzzard-62ADCC62, F.Cu at (250.8, 99.0)
- added kibuzzard-62ADCC83: G***, kibuzzard-62ADCC83, F.Cu at (258.7, 99.0)
- added kibuzzard-62ADCCBA: G***, kibuzzard-62ADCCBA, F.Cu at (261.4, 94.5)
- added kibuzzard-62ADCCBA: G***, kibuzzard-62ADCCBA, F.Cu at (247.6, 94.6)
- added kibuzzard-62ADCCCD: G***, kibuzzard-62ADCCCD, F.Cu at (261.5, 97.0)
- added kibuzzard-62ADCCCD: G***, kibuzzard-62ADCCCD, F.Cu at (247.6, 97.1)
- added kibuzzard-62ADCDD5: G***, kibuzzard-62ADCDD5, F.Cu at (254.4, 61.6)
- added kibuzzard-62ADCDEA: G***, kibuzzard-62ADCDEA, F.Cu at (256.3, 61.6)
- added kibuzzard-62ADCE22: G***, kibuzzard-62ADCE22, F.Cu at (245.9, 59.3)
- added kibuzzard-62ADCE31: G***, kibuzzard-62ADCE31, F.Cu at (247.6, 59.3)
- added kibuzzard-62ADCE43: G***, kibuzzard-62ADCE43, F.Cu at (249.2, 59.3)
- added kibuzzard-62ADCE61: G***, kibuzzard-62ADCE61, F.Cu at (242.6, 60.3)
- added kibuzzard-62ADCE79: G***, kibuzzard-62ADCE79, F.Cu at (242.7, 51.1)
- added kibuzzard-62ADCEA8: G***, kibuzzard-62ADCEA8, F.Cu at (242.6, 46.5)
- added kibuzzard-62ADD081: G***, kibuzzard-62ADD081, F.Cu at (259.0, 61.5)
- added kibuzzard-62ADD099: G***, kibuzzard-62ADD099, F.Cu at (261.7, 61.5)
- added kibuzzard-62ADD0C2: G***, kibuzzard-62ADD0C2, F.Cu at (259.2, 58.4)
- added kibuzzard-62ADD0E6: G***, kibuzzard-62ADD0E6, F.Cu at (261.9, 58.4)
- added kibuzzard-62AF803C: G***, kibuzzard-62AF803C, F.Cu at (250.8, 83.2)
- added kibuzzard-62AF804C: G***, kibuzzard-62AF804C, F.Cu at (253.5, 83.2)
- added kibuzzard-62AF8074: G***, kibuzzard-62AF8074, F.Cu at (255.9, 84.0)
- added kibuzzard-62AF8084: G***, kibuzzard-62AF8084, F.Cu at (258.6, 84.0)
- added kibuzzard-62AF8092: G***, kibuzzard-62AF8092, F.Cu at (261.2, 84.0)
- added kibuzzard-62AF80AA: G***, kibuzzard-62AF80AA, F.Cu at (245.8, 84.0)
- added kibuzzard-62AF80C4: G***, kibuzzard-62AF80C4, F.Cu at (248.2, 84.0)
- C17, C18: value 14pF -> 22pF
- J2: footprint Connector_USB:USB_Micro-B_Wuerth_614105150721_Vertical -> Connector_USB:USB_Micro-B_Amphenol_10118194_Horizontal
- J3: value Conn_01x07 -> Conn_02x04_Odd_Even; footprint Connector_PinHeader_2.54mm:PinHeader_1x07_P2.54mm_Vertical -> Connector_PinHeader_2.54mm:PinHeader_2x04_P2.54mm_Vertical
- JP1: value SolderJumper_3_Bridged12 -> SolderJumper_3_Open; footprint Jumper:SolderJumper-3_P1.3mm_Bridged12_RoundedPad1.0x1.5mm_NumberLabels -> Jumper:SolderJumper-3_P1.3mm_Open_RoundedPad1.0x1.5mm_NumberLabels
- R5, R6: value 4k7 -> 4K7
- R9: value 1K -> 604R
- Y1: value 12MHz ±30ppm 12pF 50Ω SMD-5032_2P SMD -> 12MHz ±30ppm 16pF 50Ω SMD-5032_2P SMD
- moved R15 61.9 mm to (257.3, 60.0), turned to -90 degrees
- moved C2 61.8 mm to (252.8, 47.8), turned to 180 degrees
- moved SW2 61.4 mm to (242.6, 53.5), turned to 180 degrees
- moved D5 60.8 mm to (256.3, 60.0), turned to -90 degrees
- moved R16 59.6 mm to (255.3, 60.0), turned to -90 degrees
- moved D6 58.5 mm to (254.4, 60.0), turned to -90 degrees
- moved R1 58.3 mm to (252.8, 41.7), turned to 0 degrees
- moved U1 55.1 mm to (249.2, 44.7), turned to 180 degrees
- moved C10 51.7 mm to (257.1, 64.9)
- moved C11 51.7 mm to (256.1, 64.9)
- moved C12 51.7 mm to (255.0, 64.9)
- moved C13 51.7 mm to (254.0, 64.9)
- moved C14 51.7 mm to (253.0, 64.9)
- moved C15 51.7 mm to (252.0, 64.9)
- moved C16 51.7 mm to (251.0, 64.9)
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Connections:
- J2 pad 4: Net-(J2-Pad4) -> unconnected-(J2-Pad4)
- J3 pad 1: FC_SERVO_1 -> GND
- J3 pad 2: FC_SERVO_2 -> GND
- J3 pad 3: FC_SERVO_3 -> FC_UART0_RX
- J3 pad 4: FC_SERVO_4 -> FC_UART1_RX
- J3 pad 5: FC_SERVO_5 -> FC_UART0_TX
- J3 pad 6: FC_SERVO_6 -> FC_UART1_TX
- J3 pad 7: FC_RADIO_PPM -> +5V
- J6 pad 1: Net-(J6-Pad1) -> unconnected-(J6-Pad1)
- J6 pad 8: Net-(J6-Pad8) -> unconnected-(J6-Pad8)
- U1 pad 2: Net-(U1-Pad2) -> unconnected-(U1-Pad2)
- U1 pad 3: Net-(U1-Pad3) -> unconnected-(U1-Pad3)
- U1 pad 5: Net-(U1-Pad5) -> unconnected-(U1-Pad5)
- U5 pad 12: Net-(U5-Pad12) -> unconnected-(U5-Pad12)
- U5 pad 6: Net-(U5-Pad6) -> unconnected-(U5-Pad6)
- U5 pad 7: Net-(U5-Pad7) -> unconnected-(U5-Pad7)
- U5 pad 9: Net-(U5-Pad9) -> unconnected-(U5-Pad9)
Routing:
- net +5V: track 136.2 -> 37.4 mm, vias 2 -> 1
- net FC_I2C1_SDA: track 67.7 -> 0.00 mm, vias 3 -> 0
- net FC_I2C1_SCL: track 66.2 -> 0.00 mm, vias 3 -> 0
- net GND: track 123.3 -> 68.2 mm, vias 42 -> 30
- net +3V3: track 59.6 -> 6.93 mm, vias 2 -> 0
- net FC_RUN: track 40.4 -> 5.42 mm
- net FC_UART0_RX: track 35.9 -> 1.00 mm, vias 2 -> 1
- net FC_USB_VBUS: track 32.2 -> 0.00 mm, vias 1 -> 0
- net FC_STATUS_RED: track 31.7 -> 1.13 mm, vias 3 -> 1
- net FC_SPI0_MISO: track 32.7 -> 2.42 mm
- net FC_UART0_TX: track 31.8 -> 2.44 mm, vias 2 -> 1
- net +1V1: track 36.4 -> 8.68 mm, vias 3 -> 2
- net FC_SPI0_MOSI: track 31.8 -> 4.33 mm
- net FC_SPI0_CS: track 31.0 -> 3.87 mm, vias 3 -> 1
- net FC_SPI0_SCK: track 31.9 -> 4.81 mm
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- added copper zone on In2.Cu, net +5V
- added copper zone on F.Cu, net 3V3_IO
- removed copper zone on F.Cu, net VCC
- removed copper zone on In2.Cu, net VCC
Other:
- board size 41.8 x 49.9 mm -> 30 x 65 mm
- board text removed: "3-6S"
- board text removed: "3V3"
- board text removed: "5V"
- board text removed: "BOOT"
- board text removed: "CAL"
- board text removed: "ERR"
- board text removed: "G"
- board text removed: "HERMES"
- board text removed: "Oct 2021"
- board text removed: "PPM"
- board text removed: "RDY"
- board text removed: "RESET"
- board text removed: "RX0"
- board text removed: "RX1"
- board text removed: "S1"
- board text removed: "S2"
- board text removed: "S3"
- board text removed: "S4"
- board text removed: "S5"
- board text removed: "S6"
- board text removed: "SCL1"
- board text removed: "SDA1"
- board text removed: "TX0"
- board text removed: "TX1"
- board text removed: "rayb.tech"

Commit message: more new stuff
Parts:
- removed C20: 2.2nF, Capacitor_SMD:C_0402_1005Metric_Pad0.74x0.62mm_HandSolder
- removed C22, C26: 0.1uF, Capacitor_SMD:C_0402_1005Metric_Pad0.74x0.62mm_HandSolder
- removed C25: 10nF, Capacitor_SMD:C_0402_1005Metric_Pad0.74x0.62mm_HandSolder
- removed C4: 220uF, Capacitor_SMD:CP_Elec_6.3x5.4
- removed D1: B340, Diode_SMD:D_SMC
- removed J6: Micro_SD_Card, Connector_Card:microSD_HC_Wuerth_693072010801
- removed L1: 15uH, Inductor_SMD:L_0402_1005Metric
- removed R1: 3.24k, Resistor_SMD:R_0402_1005Metric_Pad0.72x0.64mm_HandSolder
- removed R2: 10k, Resistor_SMD:R_0402_1005Metric_Pad0.72x0.64mm_HandSolder
- removed R5, R6: 4K7, Resistor_SMD:R_0402_1005Metric_Pad0.72x0.64mm_HandSolder
- removed U5: MPU-6050, Sensor_Motion:InvenSense_QFN-24_4x4mm_P0.5mm
- added C21: 2.2uF, Capacitor_SMD:C_0402_1005Metric, F.Cu at (250.9, 48.6)
- added C23: 2.2uF, Capacitor_SMD:C_0402_1005Metric, F.Cu at (250.9, 49.9)
- added C24: 47uF, Capacitor_SMD:C_0402_1005Metric, F.Cu at (254.3, 56.1)
- added C27: 47uF, Capacitor_SMD:C_0402_1005Metric, F.Cu at (254.9, 53.8)
- added C28: 100nF, Capacitor_SMD:C_0402_1005Metric, F.Cu at (245.7, 50.4)
- added C29: 100nF, Capacitor_SMD:C_0402_1005Metric, F.Cu at (248.2, 44.6)
- added C30: 10uF, Capacitor_SMD:C_0402_1005Metric, F.Cu at (248.6, 43.1)
- added C31: C_SS, Capacitor_SMD:C_0402_1005Metric, F.Cu at (253.8, 53.8)
- added C32: 100nF, Capacitor_SMD:C_0402_1005Metric, F.Cu at (250.9, 51.1)
- added D7: B340AG, Diode_SMD:D_SMB, F.Cu at (251.6, 44.1)
- added D8: MMBZ5242B, Diode_SMD:D_SOT-23_ANK, F.Cu at (246.2, 42.3)
- added L2: 8.2uH, Inductor_SMD:L_Bourns_SRP7028A_7.3x6.6mm, F.Cu at (258.4, 43.8)
- added Q1: DMP3013SFV, Package_SON:Diodes_PowerDI3333-8, F.Cu at (247.0, 47.6)
- added R10: 49.9K, Resistor_SMD:R_0402_1005Metric, F.Cu at (244.9, 55.4)
- added R11: 17.8K, Resistor_SMD:R_0402_1005Metric, F.Cu at (247.5, 58.1)
- added R17: 12K, Resistor_SMD:R_0402_1005Metric, F.Cu at (246.2, 44.6)
- added R8: 100K, Resistor_SMD:R_0402_1005Metric, F.Cu at (251.4, 58.1)
- added TP3: SPI_3V3, TestPoint:TestPoint_Pad_D1.0mm, B.Cu at (245.8, 83.8)
- added TP7: TestPoint_Small, TestPoint:TestPoint_Pad_D1.0mm, B.Cu at (260.4, 73.0)
- added TP8: TestPoint_Small, TestPoint:TestPoint_Pad_D1.0mm, B.Cu at (261.4, 65.0)
- added U6: LMR16030SDDAR, Package_SO:Texas_HSOP-8-1EP_3.9x4.9mm_P1.27mm_ThermalVias, F.Cu at (249.3, 54.5)
- C1, C2: value 10uF -> 0.1uF
- U1: value TPS5430DDAR -> BMI088; footprint TPS5430DDAR:TPS5430DDAR -> BMI088:BMI088
- moved C1 36.6 mm to (256.2, 81.1), turned to 90 degrees
- moved U1 36.4 mm to (258.6, 79.9), turned to 90 degrees
- moved C2 32.3 mm to (261.6, 78.8), turned to 90 degrees
- moved C5 4.45 mm to (260.8, 48.1), turned to 0 degrees
- moved kibuzzard-62ADCE61 2.65 mm to (244.1, 58.0), turned to 90 degrees
- moved SW2 1.66 mm to (241.8, 52.1), turned to -90 degrees
- moved kibuzzard-62ADCE79 1.65 mm to (244.1, 52.0), turned to 90 degrees
- moved C3 1.51 mm to (256.8, 48.1)
- moved kibuzzard-62ADCEA8 1.50 mm to (241.8, 45.2)
- moved P3 1.15 mm to (242.0, 47.4)
- moved P4 1.15 mm to (242.0, 43.1)
- moved U2 0.90 mm to (259.2, 53.2)
- moved SW1 0.89 mm to (241.7, 58.0), turned to 90 degrees
- moved R12 0.47 mm to (249.3, 64.3)
- moved R13 0.47 mm to (247.7, 64.3)
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Connections:
- net Net-(J2-Pad2) renamed /FCC Peripherals/d-
- net Net-(J2-Pad3) renamed /FCC Peripherals/d+
- C1 pad 1: VCC -> 3V3_IO
- C1 pad 2: GND -> Net-(C1-Pad2)
- C2 pad 2: Net-(C2-Pad2) -> 3V3_IO
- J1 pad 1: unconnected-(J1-Pad1) -> +5V
- J1 pad 10: unconnected-(J1-Pad10) -> GND
- J1 pad 19: unconnected-(J1-Pad19) -> GND
- J1 pad 26: unconnected-(J1-Pad26) -> GND
- J1 pad 29: unconnected-(J1-Pad29) -> GND
- J1 pad 3: unconnected-(J1-Pad3) -> +5V
- J1 pad 33: unconnected-(J1-Pad33) -> GND
- J1 pad 4: unconnected-(J1-Pad4) -> FC_I2C0_SDA
- J1 pad 40: unconnected-(J1-Pad40) -> GND
- J1 pad 5: unconnected-(J1-Pad5) -> GND
- J1 pad 6: unconnected-(J1-Pad6) -> FC_I2C0_SCL
- U1 pad 1: Net-(C2-Pad1) -> unconnected-(U1-Pad1)
- U1 pad 3: unconnected-(U1-Pad3) -> Net-(C1-Pad2)
- U1 pad 4: Net-(R1-Pad1) -> GND
- U1 pad 5: unconnected-(U1-Pad5) -> FC_SPI0_CS2
- U1 pad 7: VCC -> GND
- U1 pad 8: Net-(C2-Pad2) -> FC_SPI0_SCK
- U3 pad 29: FC_GPIO18 -> FC_SPI0_CS2
- U3 pad 3: FC_SPI0_CS -> FC_SPI0_CS1
Routing:
- net FC_UART0_RX: track 1.00 -> 48.7 mm
- net FC_UART0_TX: track 2.44 -> 46.9 mm
- net FC_USB_VBUS: track 0.00 -> 36.9 mm, vias 0 -> 3
- net GND: track 68.2 -> 102.4 mm, vias 30 -> 38
- net FC_BOOTSEL: track 5.19 -> 31.9 mm
- net FC_SPI0_MISO: track 2.42 -> 27.3 mm, vias 1 -> 2
- net /+12v: track 0.00 -> 24.6 mm
- net FC_SPI0_CS1: track 0.00 -> 24.1 mm, vias 0 -> 2
- net FC_RUN: track 5.42 -> 29.3 mm
- net +5V: track 37.4 -> 60.5 mm
- net FC_I2C0_SCL: track 24.1 -> 46.6 mm, vias 3 -> 1
- net +1V1: track 8.68 -> 30.2 mm, vias 2 -> 3
- net FC_I2C0_SDA: track 27.9 -> 49.3 mm, vias 3 -> 1
- net +3V3: track 6.93 -> 25.6 mm, vias 0 -> 2
- net FC_SPI0_MOSI: track 4.33 -> 22.2 mm, vias 1 -> 2
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- added copper zone on F.Cu, net /+12v
- added copper zone on B.Cu, net VCC
- removed copper zone on F.Cu, net 3V3_IO
Other:
- board text added: "JLCJLCJLCJLC"
- board text added: "TP1 - CS TP2 - MOSI TP3 - 3V3 TP4 - SCK TP5 - GND TP6 - MISO TP7 - JTG_CLK TP8 - JTG_SWD"
- board text removed: "1"
