File: Hermes/hermes_v1/hermes_v1.kicad_pcb (KiCad board)
At the start: 4 copper layers, 30 x 65 mm, 103 parts, among them J1 Conn_02x20_Odd_Even, J2 Connector_USB_B_Micro, J3 Conn_02x04_Odd_Even, J6 Micro_SD_Card, J8 Conn_01x08, J9 Conn_02x08_Odd_Even, P1 ESC1_VCC, P2 ESC1_GND, P3 LIPO_VCC, P4 LIPO_GND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

Commit message: Added VoltPak 1000
Parts:
- removed C1, C2: 10uF, Capacitor_SMD:C_0402_1005Metric_Pad0.74x0.62mm_HandSolder
- removed C4: 220uF, Capacitor_SMD:CP_Elec_6.3x5.4
- removed D1: B340, Diode_SMD:D_SMC
- removed J6: Micro_SD_Card, Connector_Card:microSD_HC_Wuerth_693072010801
- removed L1: 15uH, Inductor_SMD:L_0402_1005Metric
- removed R1: 3.24k, Resistor_SMD:R_0402_1005Metric_Pad0.72x0.64mm_HandSolder
- removed R2: 10k, Resistor_SMD:R_0402_1005Metric_Pad0.72x0.64mm_HandSolder
- removed U1: TPS5430DDAR, TPS5430DDAR:TPS5430DDAR
- added C21: 2.2uF, Capacitor_SMD:C_0402_1005Metric, F.Cu at (250.9, 48.6)
- added C23: 2.2uF, Capacitor_SMD:C_0402_1005Metric, F.Cu at (250.9, 49.9)
- added C24: 47uF, Capacitor_SMD:C_0402_1005Metric, F.Cu at (254.3, 56.1)
- added C27: 47uF, Capacitor_SMD:C_0402_1005Metric, F.Cu at (254.9, 53.8)
- added C28: 100nF, Capacitor_SMD:C_0402_1005Metric, F.Cu at (245.7, 50.4)
- added C29: 100nF, Capacitor_SMD:C_0402_1005Metric, F.Cu at (248.2, 44.6)
- added C30: 10uF, Capacitor_SMD:C_0402_1005Metric, F.Cu at (248.6, 43.1)
- added C31: C_SS, Capacitor_SMD:C_0402_1005Metric, F.Cu at (253.8, 53.8)
- added C32: 100nF, Capacitor_SMD:C_0402_1005Metric, F.Cu at (250.9, 51.1)
- added D7: B340AG, Diode_SMD:D_SMB, F.Cu at (251.6, 44.1)
- added D8: MMBZ5242B, Diode_SMD:D_SOT-23_ANK, F.Cu at (246.2, 42.3)
- added L2: 8.2uH, Inductor_SMD:L_Bourns_SRP7028A_7.3x6.6mm, F.Cu at (258.4, 43.8)
- added Q1: DMP3013SFV, Package_SON:Diodes_PowerDI3333-8, F.Cu at (247.0, 47.6)
- added R10: 49.9K, Resistor_SMD:R_0402_1005Metric, F.Cu at (244.9, 55.4)
- added R11: 17.8K, Resistor_SMD:R_0402_1005Metric, F.Cu at (247.5, 58.1)
- added R17: 12K, Resistor_SMD:R_0402_1005Metric, F.Cu at (246.2, 44.6)
- added R8: 100K, Resistor_SMD:R_0402_1005Metric, F.Cu at (251.4, 58.1)
- added TP1: SPI_CS, TestPoint:TestPoint_Pad_D1.0mm, B.Cu at (245.3, 77.2)
- added TP2: SPI_MOSI, TestPoint:TestPoint_Pad_D1.0mm, B.Cu at (248.0, 81.2)
- added TP3: SPI_3V3, TestPoint:TestPoint_Pad_D1.0mm, B.Cu at (245.8, 83.8)
- added TP4: SPI_SCK, TestPoint:TestPoint_Pad_D1.0mm, B.Cu at (246.0, 80.1)
- added TP5: SPI_GND, TestPoint:TestPoint_Pad_D1.0mm, B.Cu at (244.0, 82.5)
- added TP6: SPI_MISO, TestPoint:TestPoint_Pad_D1.0mm, B.Cu at (246.9, 75.2)
- added TP7: TestPoint_Small, TestPoint:TestPoint_Pad_D1.0mm, B.Cu at (260.4, 73.0)
- added TP8: TestPoint_Small, TestPoint:TestPoint_Pad_D1.0mm, B.Cu at (261.4, 65.0)
- added U6: LMR16030SDDAR, Package_SO:Texas_HSOP-8-1EP_3.9x4.9mm_P1.27mm_ThermalVias, F.Cu at (249.3, 54.5)
- moved C5 4.45 mm to (260.8, 48.1), turned to 0 degrees
- moved kibuzzard-62ADCE61 2.65 mm to (244.1, 58.0), turned to 90 degrees
- moved SW2 1.66 mm to (241.8, 52.1), turned to -90 degrees
- moved kibuzzard-62ADCE79 1.65 mm to (244.1, 52.0), turned to 90 degrees
- moved C3 1.51 mm to (256.8, 48.1)
- moved kibuzzard-62ADCEA8 1.50 mm to (241.8, 45.2)
- moved P3 1.15 mm to (242.0, 47.4)
- moved P4 1.15 mm to (242.0, 43.1)
- moved U2 0.90 mm to (259.2, 53.2)
- moved SW1 0.89 mm to (241.7, 58.0), turned to 90 degrees
- moved R12 0.47 mm to (249.3, 64.3)
- moved R13 0.47 mm to (247.7, 64.3)
- moved R14 0.47 mm to (246.1, 64.3)
- moved D2 0.47 mm to (249.3, 61.9)
- moved kibuzzard-62ADCE22 0.47 mm to (246.1, 59.7)
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Connections:
- net Net-(J2-Pad2) renamed /FCC Peripherals/d-
- net Net-(J2-Pad3) renamed /FCC Peripherals/d+
- J1 pad 1: unconnected-(J1-Pad1) -> +5V
- J1 pad 10: unconnected-(J1-Pad10) -> GND
- J1 pad 19: unconnected-(J1-Pad19) -> GND
- J1 pad 26: unconnected-(J1-Pad26) -> GND
- J1 pad 29: unconnected-(J1-Pad29) -> GND
- J1 pad 3: unconnected-(J1-Pad3) -> +5V
- J1 pad 33: unconnected-(J1-Pad33) -> GND
- J1 pad 40: unconnected-(J1-Pad40) -> GND
- J1 pad 5: unconnected-(J1-Pad5) -> GND
Routing:
- net FC_UART0_RX: track 1.00 -> 47.9 mm
- net FC_UART0_TX: track 2.44 -> 46.9 mm
- net GND: track 68.2 -> 111.0 mm, vias 30 -> 41
- net FC_USB_VBUS: track 0.00 -> 36.9 mm, vias 0 -> 3
- net FC_BOOTSEL: track 5.19 -> 31.9 mm
- net /+12v: track 0.00 -> 24.6 mm
- net FC_RUN: track 5.42 -> 29.3 mm
- net +5V: track 37.4 -> 60.5 mm
- net +1V1: track 8.68 -> 30.2 mm, vias 2 -> 3
- net +3V3: track 6.93 -> 25.6 mm, vias 0 -> 2
- net FC_STATUS_RED: track 1.13 -> 16.8 mm, vias 1 -> 2
- net FC_STATUS_GREEN: track 1.44 -> 15.8 mm, vias 1 -> 2
- net Net-(C32-Pad2): track 0.00 -> 13.8 mm
- net REG_5VIN: track 0.00 -> 13.7 mm, vias 0 -> 2
- net VCC: track 0.00 -> 7.95 mm
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- added copper zone on F.Cu, net /+12v
- added copper zone on B.Cu, net VCC
- removed copper zone on F.Cu, net 3V3_IO
Other:
- board text added: "JLCJLCJLCJLC"
- board text added: "TP1 - CS TP2 - MOSI TP3 - 3V3 TP4 - SCK TP5 - GND TP6 - MISO TP7 - JTG_CLK TP8 - JTG_SWD"
- board text removed: "1"
