File: Hermes/hermes_v1/_autosave-hermes_v1.kicad_pcb (KiCad board)
At the start: 4 copper layers, 32.7 x 49.9 mm, 77 parts, among them J2 Connector_USB_B_Micro, J3 Conn_01x07, J4 Conn_02x07_Odd_Even, J5 Additional IO, J6 Micro_SD_Card, J7 IO Power, P1 ESC1_VCC, P2 ESC1_GND, P3 LIPO_VCC, P4 LIPO_GND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

Commit message: new
Other:
- board text added: "HERMES"
- board text removed: "KÁRMÁN"
