File: Hermes/hermes_v1/FCC.sch (KiCad schematic (older format))
At the start: 29 parts, among them J2 FCC_BOOTSEL, J3 FCC_RESET, U1 RP2040, U4 W25Q128JVS, Y1 ABLS-12.000MHZ-B4-T

Commit message: routed rp2040
Parts:
- U1: symbol MCU_RP2040:RP2040 -> hermes_v1-rescue:RP2040-MCU_RP2040
Changed lines of the file:
@@
 $EndDescr
 $Comp
-L MCU_RP2040:RP2040 U1
+L hermes_v1-rescue:RP2040-MCU_RP2040 U1
 U 1 1 60DD7FA6
 P 3550 4900
+AR Path="/60DD7FA6" Ref="U1"  Part="1"
+AR Path="/60DD71AF/60DD7FA6" Ref="U1"  Part="1"
 F 0 "U1" H 2450 2900 50  0000 C CNN
 F 1 "RP2040" H 4500 2900 50  0000 C CNN

Commit message: new
Parts:
- removed J2: FCC_BOOTSEL, Connector_PinSocket_2.54mm:PinSocket_1x03_P2.54mm_Vertical, symbol Connector:Conn_01x03_Male
- removed J3: FCC_RESET, Connector_PinSocket_2.54mm:PinSocket_1x03_P2.54mm_Vertical, symbol Connector:Conn_01x03_Male
- added SW1: BOOT_SEL, Button_Switch_SMD:SW_SPST_PTS810, symbol Switch:SW_Push
- added SW2: RESET, Button_Switch_SMD:SW_SPST_PTS810, symbol Switch:SW_Push
- C17: renamed from C30; value 27p -> 14pF; LCSC (none) -> C458857
- C18: renamed from C31; value 27p -> 14pF; LCSC (none) -> C458857
- JP2: value FCC_3V -> MCU_EN
- U3: renamed from U1; footprint RP2040:QFN40P695X695X90-57T320N -> RP2040_minimal:RP2040-QFN-56; LCSC (none) -> C2040
- U4: LCSC (none) -> C97521
- Y1: value ABLS-12.000MHZ-B4-T -> 12MHz ±30ppm 12pF 50Ω SMD-5032_2P SMD; footprint Crystal:Crystal_SMD_HC49-SD_HandSoldering -> Crystal:Crystal_SMD_TXC_7A-2Pin_5x3.2mm; LCSC (none) -> C90884
- renumbered C16 to C10, C17 to C11, C18 to C12, C19 to C13, C20 to C14, C21 to C15, C22 to C16, C32 to C19, C12 to C6, C13 to C7, C14 to C8, C15 to C9, R15 to R10, R16 to R11, R9 to R3, R10 to R4, R2 to R5, R11 to R6, R12 to R7, R13 to R8, R14 to R9
Connections:
- net FC_GPIO26_ADC0 is gone; now on net FC_I2C1_SDA: U3.38 (GPIO26_ADC0)
- net FC_GPIO27_ADC1 is gone; now on net FC_I2C1_SCL: U3.39 (GPIO27_ADC1)
- net FC_GPIO4 is gone; now on net FC_I2C0_SDA: U3.6 (GPIO4)
- net FC_GPIO5 is gone; now on net FC_I2C0_SCL: U3.7 (GPIO5)
- net +3V3: no longer C19.1, R10.1, R11.1, R5.1, R6.1, R8.1, U4.8 (VCC)
- net FC_BOOTSEL: now also SW1.1
- net FC_I2C0_SCL: no longer U3.3 (GPIO1)
- net FC_I2C0_SDA: no longer U3.2 (GPIO0)
- net FC_RUN: now also SW2.1
- net GND: now also SW1.2, SW2.2
- net 3V_MCU: now reaches C10.1, C11.1, C12.1, C13.1, C14.1, C15.1, C16.1, C9.1, JP2.2 (B), U3.1 (IOVDD), U3.10 (IOVDD), U3.22 (IOVDD), U3.33 (IOVDD), U3.42 (IOVDD), U3.43 (ADC_AVDD), U3.44 (VREG_IN), U3.48 (USB_VDD), U3.49 (IOVDD)
- net USB-: now reaches R4.2, U3.46 (USB_DM)
- net USB+: now reaches R3.2, U3.47 (USB_DP)
- net FC_GPIO10 renamed FC_SERVO_6
- net FC_GPIO11 renamed FC_SERVO_5
- net FC_GPIO12 renamed FC_SERVO_4
- net FC_GPIO13 renamed FC_SERVO_3
- net FC_GPIO14 renamed FC_SERVO_2
- net FC_GPIO15 renamed FC_SERVO_1
- net FC_GPIO16 renamed FC_UART0_TX
- net FC_GPIO17 renamed FC_UART0_RX
- net FC_GPIO2 renamed FC_SPI0_SCK
- net FC_GPIO21 renamed FC_STATUS_RED
- net FC_GPIO22 renamed FC_STATUS_GREEN
- net FC_GPIO23 renamed FC_STATUS_BLUE
- net FC_GPIO3 renamed FC_SPI0_MOSI
- net FC_GPIO6 renamed FC_RADIO_PPM
- net FC_GPIO7 renamed FC_SERVO_7
- net FC_GPIO8 renamed FC_UART1_TX
- net FC_GPIO9 renamed FC_UART1_RX
- new net 3V3_IO: C19.1, R10.1, R11.1, R5.1, R6.1, R8.1, U4.8 (VCC)
- new net FC_SPI0_CS: U3.3 (GPIO1)
- new net FC_SPI0_MISO: U3.2 (GPIO0)
- no-connect marks 2 -> 0
Other:
- note added: "BootSel & Reset Buttons"
- note added: "Make sure C7 is close to pin 45 of RP2040"
- note added: "Make sure C9 is close to pin 44 of RP2040"
- note removed: "BOOTSEL & RESET Jumpers"
- note removed: "Make sure C13 is close to pin 45 of RP2040"
- note removed: "Make sure C15 is close to pin 44 of RP2040"

Commit message: added piUAV & Proteus_v1
Parts:
- R10, R11, R5, R6: value 4k7 -> 4K7
Changed lines of the file:
@@
 P 7650 6100
 F 0 "R6" V 7846 6100 50  0000 C CNN
-F 1 "4k7" V 7755 6100 50  0000 C CNN
+F 1 "4K7" V 7755 6100 50  0000 C CNN
 F 2 "Resistor_SMD:R_0402_1005Metric_Pad0.72x0.64mm_HandSolder" H 7650 6100 50  0001 C CNN
 F 3 "~" H 7650 6100 50  0001 C CNN
@@
 P 7650 5800
 F 0 "R5" V 7846 5800 50  0000 C CNN
-F 1 "4k7" V 7755 5800 50  0000 C CNN
+F 1 "4K7" V 7755 5800 50  0000 C CNN
 F 2 "Resistor_SMD:R_0402_1005Metric_Pad0.72x0.64mm_HandSolder" H 7650 5800 50  0001 C CNN
 F 3 "~" H 7650 5800 50  0001 C CNN
@@
 P 9450 6100
 F 0 "R11" V 9646 6100 50  0000 C CNN
-F 1 "4k7" V 9555 6100 50  0000 C CNN
+F 1 "4K7" V 9555 6100 50  0000 C CNN
 F 2 "Resistor_SMD:R_0402_1005Metric_Pad0.72x0.64mm_HandSolder" H 9450 6100 50  0001 C CNN
 F 3 "~" H 9450 6100 50  0001 C CNN
@@
 P 9450 5800
 F 0 "R10" V 9646 5800 50  0000 C CNN
-F 1 "4k7" V 9555 5800 50  0000 C CNN
+F 1 "4K7" V 9555 5800 50  0000 C CNN
 F 2 "Resistor_SMD:R_0402_1005Metric_Pad0.72x0.64mm_HandSolder" H 9450 5800 50  0001 C CNN
 F 3 "~" H 9450 5800 50  0001 C CNN
