File: Hermes/hermes_v1/FCC_Peripherals.sch (KiCad schematic (older format))
At the start: 21 parts, among them J4 5V_EXT_IN, J5 GND_EXT_IN, J6 2.54mm, J7 Conn_02x06_Odd_Even, J8 Connector_USB_B_Micro, U2 MPL3115A2, U3 MPU-6050

Commit message: changed board to pi-zero HAT design
Parts:
- removed J4: 5V_EXT_IN, TestPoint:TestPoint_Pad_2.5x2.5mm, symbol Connector:Conn_01x01_Male
- removed J5: GND_EXT_IN, TestPoint:TestPoint_Pad_D2.5mm, symbol Connector:Conn_01x01_Male
- added J1: Raspberry Pi Zero, Connector_PinHeader_2.54mm:PinHeader_2x20_P2.54mm_Vertical, symbol Connector_Generic:Conn_02x20_Odd_Even
Connections:
- net labels added: PI_5V, PI_GPIO0, PI_GPIO1, PI_GPIO10, PI_GPIO11, PI_GPIO12, PI_GPIO13, PI_GPIO14, PI_GPIO15, PI_GPIO16, PI_GPIO2, PI_GPIO21, PI_GPIO22, PI_GPIO23, PI_GPIO24, PI_GPIO25, PI_GPIO26, PI_GPIO27, PI_GPIO28, PI_GPIO29, PI_GPIO3, PI_GPIO4, PI_GPIO5, PI_GPIO6, PI_GPIO7, PI_GPIO8, PI_GPIO9
- wire segments 54 -> 83
- no-connect marks 7 -> 18
Other:
- note removed: "External 5V Solder pads"

Commit message: routed rp2040
Parts:
- J8: symbol CH330:Connector_USB_B_Micro -> hermes_v1-rescue:Connector_USB_B_Micro-CH330
Changed lines of the file:
@@
 $EndComp
 $Comp
-L CH330:Connector_USB_B_Micro J8
+L hermes_v1-rescue:Connector_USB_B_Micro-CH330 J8
 U 1 1 6103FAC5
 P 1400 6650
+AR Path="/6103FAC5" Ref="J8"  Part="1"
+AR Path="/61068FAA/6103FAC5" Ref="J8"  Part="1"
 F 0 "J8" H 1457 7117 50  0000 C CNN
 F 1 "Connector_USB_B_Micro" H 1457 7026 50  0000 C CNN

Commit message: new
Parts:
- removed BZ1: Buzzer, Buzzer_Beeper:Buzzer_TDK_PS1240P02BT_D12.2mm_H6.5mm, symbol Device:Buzzer
- removed J1: Raspberry Pi Zero, Connector_PinHeader_2.54mm:PinHeader_2x20_P2.54mm_Vertical, symbol Connector_Generic:Conn_02x20_Odd_Even
- removed J6: 2.54mm, Connector_PinSocket_2.54mm:PinSocket_1x06_P2.54mm_Vertical, symbol Connector_Generic:Conn_01x06
- removed J7: Conn_02x06_Odd_Even, Connector_PinSocket_2.54mm:PinSocket_2x06_P2.54mm_Vertical, symbol Connector_Generic:Conn_02x06_Odd_Even
- added D5, D6: LED_R, LED_SMD:LED_0402_1005Metric_Pad0.77x0.64mm_HandSolder, symbol Device:LED_Small
- added J3: Conn_01x07, Connector_PinHeader_2.54mm:PinHeader_1x07_P2.54mm_Vertical, symbol Connector_Generic:Conn_01x07
- added J4: Conn_02x07_Odd_Even, Connector_PinHeader_2.54mm:PinHeader_2x07_P2.54mm_Vertical, symbol Connector_Generic:Conn_02x07_Odd_Even
- added J5: Additional IO, Connector_PinHeader_2.54mm:PinHeader_2x03_P2.54mm_Vertical, symbol Connector_Generic:Conn_02x03_Odd_Even
- added J6: Micro_SD_Card, Connector_Card:microSD_HC_Wuerth_693072010801, symbol Connector:Micro_SD_Card
- added J7: IO Power, Connector_PinHeader_2.54mm:PinHeader_2x03_P2.54mm_Vertical, symbol Connector_Generic:Conn_02x03_Odd_Even
- added R15, R16: 33R, Resistor_SMD:R_0402_1005Metric_Pad0.72x0.64mm_HandSolder, symbol Device:R_Small
- added U7: USBLC6-2P6, Package_TO_SOT_SMD:SOT-666, symbol Power_Protection:USBLC6-2P6
- C20: renamed from C29; value 2200pf -> 2.2nF
- C22: renamed from C28; value 0.1u -> 0.1uF
- C25: renamed from C27; value 0.1u -> 10nF
- C26: value 0.1u -> 0.1uF
- J2: renamed from J8; footprint Connector_USB:USB_Mini-B_Wuerth_65100516121_Horizontal -> Connector_USB:USB_Micro-B_Wuerth_614105150721_Vertical
- renumbered C23 to C21, C24 to C23, C25 to C24, D6 to D2, D7 to D3, D8 to D4, R17 to R12, R18 to R13, R19 to R14, U3 to U5, U2 to U6
Connections:
- net +3V3: now also D5.2 (A); no longer C21.1, C23.1, C25.2, C26.1, U5.13 (VDD), U5.8 (VDDIO), U6.1 (VDD), U6.4 (VDDIO)
- net +5V: now also D6.2 (A), J4.10 (Pin_10), J4.12 (Pin_12), J4.14 (Pin_14), J4.2 (Pin_2), J4.4 (Pin_4), J4.6 (Pin_6), J4.8 (Pin_8), J7.3 (Pin_3), J7.5 (Pin_5)
- net FC_SERVO_1: now also J3.1 (Pin_1)
- net FC_SERVO_2: now also J3.2 (Pin_2)
- net FC_SERVO_3: now also J3.3 (Pin_3)
- net FC_SERVO_4: now also J3.4 (Pin_4)
- net FC_SERVO_5: now also J3.5 (Pin_5)
- net FC_SERVO_6: now also J3.6 (Pin_6)
- net FC_USB_D+: now also U7.1 (I/O1); no longer J2.3 (D+)
- net FC_USB_D-: now also U7.3 (I/O2); no longer J2.2 (D-)
- net FC_USB_VBUS: now also U7.5 (VBUS)
- net GND: now also J4.1 (Pin_1), J4.11 (Pin_11), J4.13 (Pin_13), J4.3 (Pin_3), J4.5 (Pin_5), J4.7 (Pin_7), J4.9 (Pin_9), J6.6 (VSS), J6.9 (SHIELD), J7.2 (Pin_2), J7.4 (Pin_4), J7.6 (Pin_6), R15.2, R16.2, U7.2 (GND)
- new net: J2.2 (D-), U7.4 (I/O2)
- new net: J2.3 (D+), U7.6 (I/O1)
- new net: D6.1 (K), R16.1
- new net: D5.1 (K), R15.1
- new net 3V3_IO: C21.1, C23.1, C25.2, C26.1, J6.4 (VDD), J7.1 (Pin_1), U5.13 (VDD), U5.8 (VDDIO), U6.1 (VDD), U6.4 (VDDIO)
- new net FC_I2C1_SCL: J5.1 (Pin_1)
- new net FC_I2C1_SDA: J5.2 (Pin_2)
- new net FC_RADIO_PPM: J3.7 (Pin_7)
- new net FC_SPI0_CS: J6.2 (DAT3/CD)
- new net FC_SPI0_MISO: J6.7 (DAT0)
- new net FC_SPI0_MOSI: J6.3 (CMD)
- new net FC_SPI0_SCK: J6.5 (CLK)
- new net FC_UART0_RX: J5.6 (Pin_6)
- new net FC_UART0_TX: J5.5 (Pin_5)
- new net FC_UART1_RX: J5.4 (Pin_4)
- new net FC_UART1_TX: J5.3 (Pin_3)
- no-connect marks 18 -> 9
Other:
- note added: "(7 Rows, 3 Cols, 2.54mm Pitch)"
- note added: "Additional IO"
- note added: "Micro SD Connector"
- note added: "USB Connector"
- note removed: "(3 Rows, 8 Cols, 2.54mm Pitch)"
- moved on the sheet: D2, D3, D4, J2, R12, R13, R14

Commit message: added piUAV & Proteus_v1
Parts:
- C21, C24: value 0.1u -> 0.1uF
- C23: value 10u -> 10uF
Changed lines of the file:
@@
 P 1900 5100
 F 0 "C24" H 1992 5146 50  0000 L CNN
-F 1 "0.1u" H 1992 5055 50  0000 L CNN
+F 1 "0.1uF" H 1992 5055 50  0000 L CNN
 F 2 "Capacitor_SMD:C_0402_1005Metric_Pad0.74x0.62mm_HandSolder" H 1900 5100 50  0001 C CNN
 F 3 "~" H 1900 5100 50  0001 C CNN
@@
 P 1650 4850
 F 0 "C23" H 1742 4896 50  0000 L CNN
-F 1 "10u" H 1742 4805 50  0000 L CNN
+F 1 "10uF" H 1742 4805 50  0000 L CNN
 F 2 "Capacitor_SMD:C_0402_1005Metric_Pad0.74x0.62mm_HandSolder" H 1650 4850 50  0001 C CNN
 F 3 "~" H 1650 4850 50  0001 C CNN
@@
 P 1350 4850
 F 0 "C21" H 1442 4896 50  0000 L CNN
-F 1 "0.1u" H 1442 4805 50  0000 L CNN
+F 1 "0.1uF" H 1442 4805 50  0000 L CNN
 F 2 "Capacitor_SMD:C_0402_1005Metric_Pad0.74x0.62mm_HandSolder" H 1350 4850 50  0001 C CNN
 F 3 "~" H 1350 4850 50  0001 C CNN
