File: Hermes/hermes_v1/FCC.kicad_sch (KiCad schematic)
At the start: 26 parts, among them SW1 BOOT_SEL, SW2 RESET, U3 RP2040, U4 W25Q128JVS, Y1 12MHz ±30ppm 16pF 50Ω SMD-503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

Commit message: more new stuff
Parts:
- removed R5, R6: 4K7, Resistor_SMD:R_0402_1005Metric_Pad0.72x0.64mm_HandSolder, symbol Device:R_Small
- added TP7, TP8: TestPoint_Small, TestPoint:TestPoint_Pad_D1.0mm, symbol Connector:TestPoint_Small
Connections:
- net FC_SWCLK: now also TP7.1
- net FC_SWD: now also TP8.1
- net FC_GPIO18 renamed FC_SPI0_CS2
- net FC_SPI0_CS renamed FC_SPI0_CS1
Changed lines of the file:
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@@
   (junction (at 127 55.88) (diameter 0) (color 0 0 0 0)
   )
-  (junction (at 214.63 144.145) (diameter 0) (color 0 0 0 0)
-  )
   (junction (at 134.62 45.72) (diameter 0) (color 0 0 0 0)
   )
@@
     (stroke (width 0) (type default) (color 0 0 0 0))
   )
-  (wire (pts (xy 214.63 141.605) (xy 214.63 144.145))
-    (stroke (width 0) (type default) (color 0 0 0 0))
-  )
   (wire (pts (xy 149.86 48.26) (xy 149.86 45.72))
     (stroke (width 0) (type default) (color 0 0 0 0))
@@
     (stroke (width 0) (type default) (color 0 0 0 0))
   )
-  (wire (pts (xy 223.52 144.145) (xy 214.63 144.145))
-    (stroke (width 0) (type default) (color 0 0 0 0))
-  )
   (wire (pts (xy 121.92 83.82) (xy 129.54 83.82))
     (stroke (width 0) (type default) (color 0 0 0 0))
@@
     (stroke (width 0) (type default) (color 0 0 0 0))
   )
-  (wire (pts (xy 214.63 151.765) (xy 223.52 151.765))
-    (stroke (width 0) (type default) (color 0 0 0 0))
-  )
   (polyline (pts (xy 284.48 74.93) (xy 177.8 74.93))
     (stroke (width 0) (type default) (color 0 0 0 0))
@@
     (stroke (width 0) (type default) (color 0 0 0 0))
   )
-  (wire (pts (xy 214.63 144.145) (xy 214.63 151.765))
-    (stroke (width 0) (type default) (color 0 0 0 0))
-  )
   (wire (pts (xy 165.1 55.88) (xy 165.1 57.15))
     (stroke (width 0) (type default) (color 0 0 0 0))
@@
     (stroke (width 0) (type default) (color 0 0 0 0))
   )
-  (wire (pts (xy 228.6 144.145) (xy 232.41 144.145))
-    (stroke (width 0) (type default) (color 0 0 0 0))
-  )
   (wire (pts (xy 60.96 46.99) (xy 52.07 46.99))
     (stroke (width 0) (type default) (color 0 0 0 0))
@@
   )
   (wire (pts (xy 157.48 48.26) (xy 157.48 45.72))
-    (stroke (width 0) (type default) (color 0 0 0 0))
-  )
-  (wire (pts (xy 228.6 151.765) (xy 232.41 151.765))
     (stroke (width 0) (type default) (color 0 0 0 0))
   )
@@
     )
   )
-  (global_label "FC_GPIO18" (shape input) (at 121.92 137.16 0) (fields_autoplaced)
-    (effects (font (size 1.27 1.27)) (justify left))
-    (property "Intersheet References" "${INTERSHEET_REFS}" (id 0) (at 0 0 0)
-      (effects (font (size 1.27 1.27)) hide)
-    )
-  )
   (global_label "FC_QSPI_SD3" (shape input) (at 251.46 49.53 0) (fields_autoplaced)
     (effects (font (size 1.27 1.27)) (justify left))
@@
     )
   )
-  (global_label "3V3_IO" (shape input) (at 214.63 141.605 0) (fields_autoplaced)
-    (effects (font (size 1.27 1.27)) (justify left))
-    (property "Intersheet References" "${INTERSHEET_REFS}" (id 0) (at 31.75 -3.175 0)
-      (effects (font (size 1.27 1.27)) hide)
-    )
-  )
   (global_label "FC_USB_D+" (shape input) (at 137.16 76.2 0) (fields_autoplaced)
     (effects (font (size 1.27 1.27)) (justify left))
@@
     )
   )
+  (global_label "FC_SWD" (shape input) (at 44.45 184.785 180) (fields_autoplaced)
+    (effects (font (size 1.27 1.27)) (justify right))
+    (property "Intersheet References" "${INTERSHEET_REFS}" (id 0) (at -13.97 26.035 0)
+      (effects (font (size 1.27 1.27)) hide)
+    )
+  )
   (global_label "FC_RUN" (shape input) (at 58.42 144.78 180) (fields_autoplaced)
     (effects (font (size 1.27 1.27)) (justify right))
@@
     )
   )
+  (global_label "FC_SPI0_CS2" (shape input) (at 121.92 137.16 0) (fields_autoplaced)
+    (effects (font (size 1.27 1.27)) (justify left))
+    (property "Intersheet References" "${INTERSHEET_REFS}" (id 0) (at 136.5209 137.0806 0)
+      (effects (font (size 1.27 1.27)) (justify left) hide)
+    )
+  )
   (global_label "FC_STATUS_GREEN" (shape input) (at 121.92 147.32 0) (fields_autoplaced)
     (effects (font (size 1.27 1.27)) (justify left))
@@
     )
   )
+  (global_label "FC_SWCLK" (shape input) (at 44.45 178.435 180) (fields_autoplaced)
+    (effects (font (size 1.27 1.27)) (justify right))
+    (property "Intersheet References" "${INTERSHEET_REFS}" (id 0) (at -13.97 22.225 0)
+      (effects (font (size 1.27 1.27)) hide)
+    )
+  )
   (global_label "FC_UART1_TX" (shape input) (at 121.92 111.76 0) (fields_autoplaced)
     (effects (font (size 1.27 1.27)) (justify left))
@@
     )
   )
-  (global_label "FC_I2C0_SDA" (shape input) (at 232.41 151.765 0) (fields_autoplaced)
-    (effects (font (size 1.27 1.27)) (justify left))
-    (property "Intersheet References" "${INTERSHEET_REFS}" (id 0) (at 31.75 -3.175 0)
-      (effects (font (size 1.27 1.27)) hide)
-    )
-  )
   (global_label "FC_SERVO_2" (shape input) (at 121.92 127 0) (fields_autoplaced)
     (effects (font (size 1.27 1.27)) (justify left))
@@
     )
   )
-  (global_label "FC_SPI0_CS" (shape input) (at 121.92 93.98 0) (fields_autoplaced)
-    (effects (font (size 1.27 1.27)) (justify left))
-    (property "Intersheet References" "${INTERSHEET_REFS}" (id 0) (at 0 0 0)
-      (effects (font (size 1.27 1.27)) hide)
+  (global_label "FC_SPI0_CS1" (shape input) (at 121.92 93.98 0) (fields_autoplaced)
+    (effects (font (size 1.27 1.27)) (justify left))
+    (property "Intersheet References" "${INTERSHEET_REFS}" (id 0) (at 136.5209 93.9006 0)
+      (effects (font (size 1.27 1.27)) (justify left) hide)
     )
   )
@@
     (effects (font (size 1.27 1.27)) (justify left))
     (property "Intersheet References" "${INTERSHEET_REFS}" (id 0) (at 0 0 0)
-      (effects (font (size 1.27 1.27)) hide)
-    )
-  )
-  (global_label "FC_I2C0_SCL" (shape input) (at 232.41 144.145 0) (fields_autoplaced)
-    (effects (font (size 1.27 1.27)) (justify left))
-    (property "Intersheet References" "${INTERSHEET_REFS}" (id 0) (at 31.75 -3.175 0)
       (effects (font (size 1.27 1.27)) hide)
     )
@@
     (pin "1")
   )
-  (symbol (lib_id "Device:R_Small") (at 226.06 151.765 90) (unit 1)
-    (in_bom yes) (on_board yes)
-    (property "Reference" "R6" (id 0) (at 226.06 146.7866 90))
-    (property "Value" "4K7" (id 1) (at 226.06 149.098 90))
-    (property "Footprint" "Resistor_SMD:R_0402_1005Metric_Pad0.72x0.64mm_HandSolder" (id 2) (at 226.06 151.765 0)
-      (effects (font (size 1.27 1.27)) hide)
-    )
-    (property "Datasheet" "~" (id 3) (at 226.06 151.765 0)
-      (effects (font (size 1.27 1.27)) hide)
-    )
-    (pin "1")
-    (pin "2")
-  )
-  (symbol (lib_id "Device:R_Small") (at 226.06 144.145 90) (unit 1)
-    (in_bom yes) (on_board yes)
-    (property "Reference" "R5" (id 0) (at 226.06 139.1666 90))
-    (property "Value" "4K7" (id 1) (at 226.06 141.478 90))
-    (property "Footprint" "Resistor_SMD:R_0402_1005Metric_Pad0.72x0.64mm_HandSolder" (id 2) (at 226.06 144.145 0)
-      (effects (font (size 1.27 1.27)) hide)
-    )
-    (property "Datasheet" "~" (id 3) (at 226.06 144.145 0)
-      (effects (font (size 1.27 1.27)) hide)
-    )
-    (pin "1")
-    (pin "2")
-  )
   (symbol (lib_id "power:GND") (at 217.17 90.17 90) (unit 1)
     (in_bom yes) (on_board yes)
@@
     (pin "2")
   )
+  (symbol (lib_id "Connector:TestPoint_Small") (at 44.45 178.435 0) (unit 1)
+    (in_bom yes) (on_board yes) (fields_autoplaced)
+    (property "Reference" "TP7" (id 0) (at 45.593 177.5265 0)
+      (effects (font (size 1.27 1.27)) (justify left))
+    )
+    (property "Value" "TestPoint_Small" (id 1) (at 45.593 180.3016 0)
+      (effects (font (size 1.27 1.27)) (justify left))
+    )
+    (property "Footprint" "TestPoint:TestPoint_Pad_D1.0mm" (id 2) (at 49.53 178.435 0)
+      (effects (font (size 1.27 1.27)) hide)
+    )
+    (property "Datasheet" "~" (id 3) (at 49.53 178.435 0)
+      (effects (font (size 1.27 1.27)) hide)
+    )
+    (pin "1")
+  )
+  (symbol (lib_id "Connector:TestPoint_Small") (at 44.45 184.785 0) (unit 1)
+    (in_bom yes) (on_board yes) (fields_autoplaced)
+    (property "Reference" "TP8" (id 0) (at 45.593 183.8765 0)
+      (effects (font (size 1.27 1.27)) (justify left))
+    )
+    (property "Value" "TestPoint_Small" (id 1) (at 45.593 186.6516 0)
+      (effects (font (size 1.27 1.27)) (justify left))
+    )
+    (property "Footprint" "TestPoint:TestPoint_Pad_D1.0mm" (id 2) (at 49.53 184.785 0)
+      (effects (font (size 1.27 1.27)) hide)
+    )
+    (property "Datasheet" "~" (id 3) (at 49.53 184.785 0)
+      (effects (font (size 1.27 1.27)) hide)
+    )
+    (pin "1")
+  )
 )
