File: Hermes/hermes_v1/FCC_Peripherals.kicad_sch (KiCad schematic)
At the start: 22 parts, among them J1 Conn_02x20_Odd_Even, J2 Connector_USB_B_Micro, J3 Conn_02x04_Odd_Even, J6 Micro_SD_Card, J8 Conn_01x08, J9 Conn_02x08_Odd_Even, U5 MPU-6050, U7 USBLC6-2P6

Commit message: more new stuff
Parts:
- removed C20: 2.2nF, Capacitor_SMD:C_0402_1005Metric_Pad0.74x0.62mm_HandSolder, symbol Device:C_Small
- removed C22, C26: 0.1uF, Capacitor_SMD:C_0402_1005Metric_Pad0.74x0.62mm_HandSolder, symbol Device:C_Small
- removed C25: 10nF, Capacitor_SMD:C_0402_1005Metric_Pad0.74x0.62mm_HandSolder, symbol Device:C_Small
- removed J6: Micro_SD_Card, Connector_Card:microSD_HC_Wuerth_693072010801, symbol Connector:Micro_SD_Card
- removed U5: MPU-6050, Sensor_Motion:InvenSense_QFN-24_4x4mm_P0.5mm, symbol Sensor_Motion:MPU-6050
- added C1, C2: 0.1uF, Capacitor_SMD:C_0402_1005Metric_Pad0.74x0.62mm_HandSolder, symbol Device:C_Small
- added U1: BMI088, BMI088:BMI088, symbol BMI088:BMI088
Connections:
- net +5V: now also J1.1 (Pin_1), J1.3 (Pin_3)
- net 3V3_IO: now also C1.1, C2.2
- net FC_I2C0_SCL: now also J1.6 (Pin_6)
- net FC_I2C0_SDA: now also J1.4 (Pin_4)
- net FC_SPI0_MISO: now also U1.10 (SDO2), U1.15 (SDO1)
- net FC_SPI0_MOSI: now also U1.9 (SDA/SDI)
- net FC_SPI0_SCK: now also U1.8 (SCL/SCK)
- net GND: now also J1.10 (Pin_10), J1.19 (Pin_19), J1.26 (Pin_26), J1.29 (Pin_29), J1.33 (Pin_33), J1.40 (Pin_40), J1.5 (Pin_5), U1.2 (NC), U1.4 (GNDA), U1.6 (GNDIO), U1.7 (PS)
- net d-: now reaches J2.2 (D-), U7.4 (I/O2)
- net d+: now reaches J2.3 (D+), U7.6 (I/O1)
- new net: C2.1, U1.11 (VDDIO)
- new net: C1.2, U1.3 (VDD)
- new net FC_SPI0_CS1: U1.14 (CSB1)
- new net FC_SPI0_CS2: U1.5 (CSB2)
- no-connect marks 7 -> 5
Other:
- note added: "SPI JUMPERS"
- note removed: "Assign proper labels to suitable I2C0 pins on FCC"
- note removed: "Inertial Measurement Unit"
- note removed: "Micro SD Connector"
