File: Hermes_Pico/Hermes_Pico/Hermes_Pico.kicad_pcb (KiCad board)
At the start: 2 copper layers, 53 x 65 mm, 22 parts, among them J1 Conn_01x08, J2 Conn_02x20_Odd_Even, J3 Conn_02x08_Odd_Even, J4 Micro_SD_Card, J5 GPS_HEADER, J6 RESET_HEADER, J7 SWD_DEBUG, U1 Pico, U2 MPU-6050, U3 MPL3115A2

Commit message: new
Parts:
- added R1: R_Small, Resistor_SMD:R_0402_1005Metric, F.Cu at (251.8, 80.0)
- added R2: R_Small, Resistor_SMD:R_0402_1005Metric, F.Cu at (251.8, 78.7)
- added R3: R_Small, Resistor_SMD:R_0402_1005Metric, F.Cu at (240.7, 71.0)
- added R4: R_Small, Resistor_SMD:R_0402_1005Metric, F.Cu at (240.6, 73.7)
- moved C4 99.8 mm to (243.6, 118.5), turned to 90 degrees
- moved C1 99.7 mm to (237.3, 115.9), turned to 270 degrees
- moved C2 97.3 mm to (238.5, 120.3), turned to 180 degrees
- moved C3 89.6 mm to (237.3, 117.9), turned to 90 degrees
- moved C6 86.7 mm to (233.4, 119.7), turned to 90 degrees
- moved C7 84.3 mm to (233.8, 115.4)
- moved C5 81.2 mm to (233.9, 118.1)
- moved REF** 1.74 mm to (256.2, 116.7)
Routing:
- net FC_I2C0_SCL: track 0.00 -> 77.8 mm, vias 0 -> 4
- net FC_I2C0_SDA: track 0.00 -> 75.9 mm, vias 0 -> 4
- net +3V3: track 106.5 -> 174.3 mm, vias 0 -> 4
- net GND: track 26.9 -> 44.6 mm, vias 5 -> 12
- net FC_I2C1_SCL: track 14.2 -> 17.7 mm, vias 0 -> 1
- net Net-(C5-Pad1): track 0.00 -> 1.47 mm
- net Net-(C4-Pad2): track 0.00 -> 1.27 mm
- net Net-(C3-Pad2): track 0.00 -> 1.25 mm
- net FC_I2C1_SDA: track 21.3 -> 22.2 mm
Other:
- board text added: "rayb.tech"
