File: Hermes_Pico/Hermes_Pico/Hermes_Pico.sch (KiCad schematic (older format))
At the start: 21 parts, among them J1 Conn_01x08, J2 Conn_02x20_Odd_Even, J3 Conn_02x08_Odd_Even, J4 Micro_SD_Card, J5 GPS_HEADER, J6 RESET_HEADER, J7 SWD_DEBUG, U1 Pico, U2 MPU-6050, U3 MPL3115A2

Commit message: new
Parts:
- added R1, R2, R3, R4: R_Small, Resistor_SMD:R_0402_1005Metric, symbol Device:R_Small
- C1: value 0.1uF -> 10nF; LCSC (none) -> C15195
- C2, C3, C5, C7: LCSC (none) -> C307331
- C4: value 2200pF -> 2.2nF; LCSC (none) -> C1531
- C6: LCSC (none) -> C15525
- J4: LCSC (none) -> C164170
- U2: LCSC (none) -> C24112
Connections:
- net +3V3: now also R1.2, R2.1, R3.2, R4.1
- net FC_I2C0_SCL: now also R4.2
- net FC_I2C0_SDA: now also R3.1
- net FC_I2C1_SCL: now also R2.2
- net FC_I2C1_SDA: now also R1.1
- no-connect marks 40 -> 50
Changed lines of the file:
@@
 F 2 "Connector_Card:microSD_HC_Wuerth_693072010801" H 10100 2000 50  0001 C CNN
 F 3 "http://katalog.we-online.de/em/datasheet/693072010801.pdf" H 8950 1700 50  0001 C CNN
+F 4 "C164170" H 8950 1700 50  0001 C CNN "LCSC"
 	1    8950 1700
 	1    0    0    -1
@@
 F 2 "Sensor_Motion:InvenSense_QFN-24_4x4mm_P0.5mm" H 1800 5350 50  0001 C CNN
 F 3 "https://store.invensense.com/datasheets/invensense/MPU-6050_DataSheet_V3%204.pdf" H 1800 6000 50  0001 C CNN
+F 4 "C24112" H 1800 6150 50  0001 C CNN "LCSC"
 	1    1800 6150
 	1    0    0    -1
@@
 F 2 "Capacitor_SMD:C_0402_1005Metric" H 2650 6550 50  0001 C CNN
 F 3 "~" H 2650 6550 50  0001 C CNN
+F 4 "C307331" H 2650 6550 50  0001 C CNN "LCSC"
 	1    2650 6550
 	-1   0    0    1
@@
 P 2800 6450
 F 0 "C4" H 2708 6404 50  0000 R CNN
-F 1 "2200pF" H 2708 6495 50  0000 R CNN
+F 1 "2.2nF" H 2708 6495 50  0000 R CNN
 F 2 "Capacitor_SMD:C_0402_1005Metric" H 2800 6450 50  0001 C CNN
 F 3 "~" H 2800 6450 50  0001 C CNN
+F 4 "C1531" H 2800 6450 50  0001 C CNN "LCSC"
 	1    2800 6450
 	-1   0    0    1
@@
 F 2 "Capacitor_SMD:C_0402_1005Metric" H 2000 5350 50  0001 C CNN
 F 3 "~" H 2000 5350 50  0001 C CNN
+F 4 "C307331" V 2000 5350 50  0001 C CNN "LCSC"
 	1    2000 5350
 	0    -1   -1   0
@@
 P 1600 5350
 F 0 "C1" V 1800 5450 50  0000 C CNN
-F 1 "0.1uF" V 1700 5450 50  0000 C CNN
+F 1 "10nF" V 1700 5450 50  0000 C CNN
 F 2 "Capacitor_SMD:C_0402_1005Metric" H 1600 5350 50  0001 C CNN
 F 3 "~" H 1600 5350 50  0001 C CNN
+F 4 "C15195" V 1600 5350 50  0001 C CNN "LCSC"
 	1    1600 5350
 	0    -1   -1   0
@@
 F 2 "Capacitor_SMD:C_0402_1005Metric" H 2550 1300 50  0001 C CNN
 F 3 "~" H 2550 1300 50  0001 C CNN
+F 4 "C15525" H 2550 1300 50  0001 C CNN "LCSC"
 	1    2550 1300
 	-1   0    0    1
@@
 F 2 "Capacitor_SMD:C_0402_1005Metric" H 2750 1300 50  0001 C CNN
 F 3 "~" H 2750 1300 50  0001 C CNN
+F 4 "C307331" H 2750 1300 50  0001 C CNN "LCSC"
 	1    2750 1300
 	1    0    0    -1
@@
 F 2 "Capacitor_SMD:C_0402_1005Metric" H 2150 1800 50  0001 C CNN
 F 3 "~" H 2150 1800 50  0001 C CNN
+F 4 "C307331" H 2150 1800 50  0001 C CNN "LCSC"
 	1    2150 1800
 	1    0    0    -1
@@
 Text GLabel 4400 4600 2    50   Input ~ 0
 FC_UART0_TX
+Text GLabel 5550 3250 0    50   Input ~ 0
+FC_I2C1_SCL
+Text GLabel 5550 3150 0    50   Input ~ 0
+FC_I2C1_SDA
+Text GLabel 6900 3150 0    50   Input ~ 0
+FC_I2C0_SDA
+Text GLabel 6900 3250 0    50   Input ~ 0
+FC_I2C0_SCL
+$Comp
+L Device:R_Small R2
+U 1 1 61620B72
+P 5750 3250
+F 0 "R2" V 5950 3250 50  0000 C CNN
+F 1 "R_Small" V 5850 3250 50  0000 C CNN
+F 2 "Resistor_SMD:R_0402_1005Metric" H 5750 3250 50  0001 C CNN
+F 3 "~" H 5750 3250 50  0001 C CNN
+F 4 "C25900" V 5750 3250 50  0001 C CNN "LCSC"
+	1    5750 3250
+	0    1    1    0
+$EndComp
+$Comp
+L Device:R_Small R1
+U 1 1 61625668
+P 5750 3150
+F 0 "R1" V 5950 3150 50  0000 C CNN
+F 1 "R_Small" V 5850 3150 50  0000 C CNN
+F 2 "Resistor_SMD:R_0402_1005Metric" H 5750 3150 50  0001 C CNN
+F 3 "~" H 5750 3150 50  0001 C CNN
+F 4 "C25900" V 5750 3150 50  0001 C CNN "LCSC"
+	1    5750 3150
+	0    -1   -1   0
+$EndComp
+Wire Wire Line
+	5550 3150 5650 3150
+Wire Wire Line
+	5550 3250 5650 3250
+$Comp
+L power:+3.3V #PWR030
+U 1 1 6162D675
+P 5950 3250
+F 0 "#PWR030" H 5950 3100 50  0001 C CNN
+F 1 "+3.3V" V 5965 3378 50  0000 L CNN
+F 2 "" H 5950 3250 50  0001 C CNN
+F 3 "" H 5950 3250 50  0001 C CNN
+	1    5950 3250
+	0    1    1    0
+$EndComp
+$Comp
+L power:+3.3V #PWR029
+U 1 1 6162E610
+P 5950 3150
+F 0 "#PWR029" H 5950 3000 50  0001 C CNN
+F 1 "+3.3V" V 5965 3278 50  0000 L CNN
+F 2 "" H 5950 3150 50  0001 C CNN
+F 3 "" H 5950 3150 50  0001 C CNN
+	1    5950 3150
+	0    1    1    0
+$EndComp
+Wire Wire Line
+	5950 3150 5850 3150
+Wire Wire Line
+	5850 3250 5950 3250
+$Comp
+L Device:R_Small R4
+U 1 1 61637EF6
+P 7100 3250
+F 0 "R4" V 7300 3250 50  0000 C CNN
+F 1 "R_Small" V 7200 3250 50  0000 C CNN
+F 2 "Resistor_SMD:R_0402_1005Metric" H 7100 3250 50  0001 C CNN
+F 3 "~" H 7100 3250 50  0001 C CNN
+F 4 "C25900" V 7100 3250 50  0001 C CNN "LCSC"
+	1    7100 3250
+	0    1    1    0
+$EndComp
+$Comp
+L Device:R_Small R3
+U 1 1 61637F00
+P 7100 3150
+F 0 "R3" V 7300 3150 50  0000 C CNN
+F 1 "R_Small" V 7200 3150 50  0000 C CNN
+F 2 "Resistor_SMD:R_0402_1005Metric" H 7100 3150 50  0001 C CNN
+F 3 "~" H 7100 3150 50  0001 C CNN
+F 4 "C25900" V 7100 3150 50  0001 C CNN "LCSC"
+	1    7100 3150
+	0    -1   -1   0
+$EndComp
+Wire Wire Line
+	6900 3150 7000 3150
+Wire Wire Line
+	6900 3250 7000 3250
+$Comp
+L power:+3.3V #PWR032
+U 1 1 61637F0C
+P 7300 3250
+F 0 "#PWR032" H 7300 3100 50  0001 C CNN
+F 1 "+3.3V" V 7315 3378 50  0000 L CNN
+F 2 "" H 7300 3250 50  0001 C CNN
+F 3 "" H 7300 3250 50  0001 C CNN
+	1    7300 3250
+	0    1    1    0
+$EndComp
+$Comp
+L power:+3.3V #PWR031
+U 1 1 61637F16
+P 7300 3150
+F 0 "#PWR031" H 7300 3000 50  0001 C CNN
+F 1 "+3.3V" V 7315 3278 50  0000 L CNN
+F 2 "" H 7300 3150 50  0001 C CNN
+F 3 "" H 7300 3150 50  0001 C CNN
+	1    7300 3150
+	0    1    1    0
+$EndComp
+Wire Wire Line
+	7300 3150 7200 3150
+Wire Wire Line
+	7200 3250 7300 3250
+NoConn ~ 4400 2800
+NoConn ~ 4400 3000
+NoConn ~ 4400 3200
+NoConn ~ 4400 3300
+NoConn ~ 4400 3400
+NoConn ~ 4400 3800
+NoConn ~ 4400 4000
+NoConn ~ 4400 4100
+NoConn ~ 4400 4200
+NoConn ~ 4400 4300
 $EndSCHEMATC
