File: Proteus/proteus_v1/proteus_v1.kicad_pcb (KiCad board)
At the start: 2 copper layers, 36 parts, among them J1 Connector_USB_B_Micro, P1 LIPO_VCC, P2 LIPO_GND, P3 ESC1_VCC, P4 ESC1_GND, P5 ESC2_VCC, P6 ESC2_GND, U1 LMR16030SDDAR, U2 LD1117S33TR_SOT223, U3 USBLC6-2P6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

Commit message: Added initial voltage circuit
Parts:
- added C6: 2.2nF, Capacitor_SMD:C_0402_1005Metric_Pad0.74x0.62mm_HandSolder, F.Cu at (134.7, 72.6)
- added C7: 0.1uF, Capacitor_SMD:C_0402_1005Metric_Pad0.74x0.62mm_HandSolder, F.Cu at (131.5, 74.6)
- added C8: 10nF, Capacitor_SMD:C_0402_1005Metric_Pad0.74x0.62mm_HandSolder, F.Cu at (131.5, 76.5)
- added C9: 0.1uF, Capacitor_SMD:C_0402_1005Metric_Pad0.74x0.62mm_HandSolder, F.Cu at (131.5, 72.6)
- added U5: MPU-6050, Sensor_Motion:InvenSense_QFN-24_4x4mm_P0.5mm, F.Cu at (126.7, 74.8)
