File: Proteus/proteus_v1/proteus_v1.kicad_sch (KiCad schematic)
At the start: 36 parts, among them J1 Connector_USB_B_Micro, P1 LIPO_VCC, P2 LIPO_GND, P3 ESC1_VCC, P4 ESC1_GND, P5 ESC2_VCC, P6 ESC2_GND, U1 LMR16030SDDAR, U2 LD1117S33TR_SOT223, U3 USBLC6-2P6, U4 MIMXRT1062DVL6A

Commit message: Added initial voltage circuit
Parts:
- removed U3: USBLC6-2P6, Package_TO_SOT_SMD:SOT-666, symbol Power_Protection:USBLC6-2P6
- added C6: 2.2nF, Capacitor_SMD:C_0402_1005Metric_Pad0.74x0.62mm_HandSolder, symbol Device:C_Small
- added C7, C9: 0.1uF, Capacitor_SMD:C_0402_1005Metric_Pad0.74x0.62mm_HandSolder, symbol Device:C_Small
- added C8: 10nF, Capacitor_SMD:C_0402_1005Metric_Pad0.74x0.62mm_HandSolder, symbol Device:C_Small
- added C?: 2.2uF, symbol Device:C_Small
- added C? (x2): 4.7uF, symbol Device:C_Small
- added C? (x4): 0.22uF, symbol Device:C_Small
- added C?: 0.22, symbol Device:C_Small
- added C?: 10nF, symbol Device:C_Small
- added C?: 10uF, symbol Device:C_Small
- added JP?: MCU_5V, Jumper:SolderJumper-2_P1.3mm_Open_RoundedPad1.0x1.5mm, symbol Jumper:SolderJumper_2_Open
- added L?: 120, symbol Device:L_Ferrite_Small
- added Q?: DMG2305UX, Package_TO_SOT_SMD:SOT-23, symbol Transistor_FET:DMG2301L
- added R?: 100K, symbol Device:R_Small
- added U5: MPU-6050, Sensor_Motion:InvenSense_QFN-24_4x4mm_P0.5mm, symbol Sensor_Motion:MPU-6050
- added U?: TLV75733PDRV, Package_SON:WSON-6-1EP_2x2mm_P0.65mm_EP1x1.6mm, symbol Regulator_Linear:TLV75733PDRV
Connections:
- net +3V3: no longer C4.1, JP2.1 (A), U2.2 (VO)
- net 3V3_IO: now also C8.2, C9.1, U5.13 (VDD), U5.8 (VDDIO)
- net GND: now also C6.2, C7.2, C8.1, C9.2, C?.1, C?.1, C?.2, C?.2, C?.2, C?.2, C?.2, C?.2, C?.2, C?.2, Q?.1 (G), U5.1 (CLKIN), U5.11 (FSYNC), U5.18 (GND), U?.3 (GND), U?.7 (GND)
- net 3V3_MCU: now reaches U4.E6 (NVCC_EMC), U4.F5 (NVCC_EMC)
- net 3V3_MCU: now also U4.E9 (NVCC_GPIO), U4.F10 (NVCC_GPIO), U4.J10 (NVCC_GPIO), U4.J6 (NVCC_SD0), U4.K4 (DCDC_IN_Q), U4.K5 (NVCC_SD1), U4.N14 (VDDA_ADC_3P3), U4.P12 (VDD_HIGH_IN), C?.1, C?.1, C?.1, C?.1, R?.1, U?.1 (OUT)
- net at U4.K7 (PMIC_ON_REQ): now also R?.2, U?.4 (EN)
- net at U4.L1 (DCDC_IN), U4.L2 (DCDC_IN): now also C?.1, C?.1, C?.1, L?.1
- net 5VBUS: now reaches U4.N6 (USB_OTG1_VBUS)
- net 5VBUS: now also U4.P6 (USB_OTG2_VBUS), C?.2, C?.2, JP?.1 (A), Q?.2 (S), U?.6 (IN)
- net REG_5VIN renamed REG_5VOUT
- net REG_5VOUT: now also C?.1, JP?.2 (B), Q?.3 (D)
- new net: C7.1, U5.10 (REGOUT)
- new net: C6.1, U5.20 (CPOUT)
- new net: C4.1, JP2.1 (A), U2.2 (VO)
- new net FC_I2C0_SCL: U5.23 (SCL)
- new net FC_I2C0_SDA: U5.24 (SDA)
- no-connect marks 2 -> 6
Other:
- note added: "Assign proper labels to suitable I2C0 pins on FCC"
- note added: "IMU"
- note removed: "IO 3.3V Enable Jumper (verify nominal IO voltage before bridging)"
- note removed: "USB"
- moved on the sheet: C2, C4, D2, D3, D4, D5, D6, J1, JP1, JP2, P3, P4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
