File: VoltPak-1000/VolPak-1000/VolPak-1000.kicad_pcb (KiCad board)
At the start: 4 copper layers, 153.7 x 108.5 mm, 185 parts, among them J1 USB_C_Receptacle_USB2.0_14P, J10 UART JST, J11 USB_A, J12 USB_C_Receptacle_USB2.0_14P, J2 SPI JST, J3 Input Switch, J4 12V Battery Input, J5 Fan Connector, J6 AC Outlet, J7 EGS002, J8 I2C JST, J9 POWER JST, Q1 SS8050, Q10 FGH40N65, Q11 FGH40N65, Q12 S8050, Q13 S8050, Q2 SS8050, Q3 IRF3205, Q4 IRF3205, Q5 IRF3205, Q6 IRF3205, Q7 SS8050, Q8 FGH40N65, Q9 FGH40N65, SW1 SW_Push, SW2 SW_Push, SW4 SW_Push, SW5 SW_Push, T1 E55, U1 ESP32-S3, U10 AP63203WU, U11 AP63205WU, U2 W25Q128JVS, U3 CP2102N-Axx-xQFN28, U4 LD1117S18TR_SOT223, U5 SG3525, U6 L7812, U7 L7805, U8 INA219BxDCN, U9 INA219BxDCN, Y1 40MHz +/-10PPM 8pF

Commit message: completed layout
Parts:
- added REF**: MountingHole_3.5mm_Pad_TopBottom, MountingHole:MountingHole_3.5mm_Pad_TopBottom, F.Cu at (70.3, 52.3)
- added REF**: MountingHole_3.5mm_Pad_TopBottom, MountingHole:MountingHole_3.5mm_Pad_TopBottom, F.Cu at (203.9, 52.3)
- added REF**: MountingHole_3.5mm_Pad_TopBottom, MountingHole:MountingHole_3.5mm_Pad_TopBottom, F.Cu at (203.7, 140.7)
- added REF**: MountingHole_3.5mm_Pad_TopBottom, MountingHole:MountingHole_3.5mm_Pad_TopBottom, F.Cu at (70.1, 140.7)
- C40: footprint Capacitor_THT:C_Disc_D4.3mm_W1.9mm_P5.00mm -> Capacitor_SMD:C_2220_5750Metric_Pad1.97x5.40mm_HandSolder
- C41, C42: footprint Capacitor_SMD:C_0603_1608Metric -> Capacitor_SMD:C_2220_5750Metric_Pad1.97x5.40mm_HandSolder
- CHOKE1: value 2.5MH 10A -> 2MH 10A
- L5: footprint Inductor_SMD:L_0402_1005Metric -> Inductor_SMD:L_0603_1608Metric
- R38, R39: footprint Resistor_SMD:R_0815_2038Metric -> Resistor_SMD:R_2512_6332Metric
- moved C40 13.4 mm to (200.2, 63.2), turned to -90 degrees
- moved T1 9.88 mm to (86.9, 97.2)
- moved U6 6.39 mm to (147.3, 118.7), turned to 180 degrees
- moved U7 5.42 mm to (158.8, 118.7), turned to 180 degrees
- moved Q3 5.34 mm to (105.5, 105.7), turned to 180 degrees
- moved Q6 5.25 mm to (94.4, 105.7), turned to 180 degrees
- moved Q5 5.14 mm to (83.3, 105.7), turned to 180 degrees
- moved Q4 5.07 mm to (116.6, 105.7), turned to 180 degrees
- moved R38 3.42 mm to (78.2, 132.6), turned to 90 degrees
- moved C42 2.41 mm to (195.1, 46.0)
- moved C41 2.36 mm to (160.5, 45.7)
- moved L5 0.66 mm to (140.4, 128.0)
- moved R39 0.50 mm to (78.2, 140.5), turned to -90 degrees
Connections:
- D18 pad 2: Net-(T1-OUT2B) -> Net-(T1-AUX+)
- D18 pad 3: Net-(T1-OUT2A) -> Net-(T1-NC16)
- T1 pad 10: (no net) -> INV_TR-
- T1 pad 11: (no net) -> INV_TR-
- T1 pad 12: (no net) -> 18VAC+
- T1 pad 13: (no net) -> 18VAC-
- T1 pad 14: (no net) -> unconnected-(T1-NC14-Pad14)
- T1 pad 2: +BATT -> INV_TR+
- T1 pad 3: INV_TR- -> INV_TR+
- T1 pad 4: 18VAC+ -> unconnected-(T1-NC4-Pad4)
- T1 pad 5: 18VAC- -> +BATT
- T1 pad 6: Net-(T1-OUT2A) -> +BATT
- T1 pad 7: Net-(T1-OUT2B) -> +BATT
- T1 pad 8: (no net) -> unconnected-(T1-NC8-Pad8)
- T1 pad 9: (no net) -> INV_TR-
Routing:
- net INV_TR-: track 59.9 -> 134.6 mm, vias 0 -> 1
- net Net-(T1-AUX+): track 0.00 -> 63.2 mm
- net Net-(T1-NC16): track 0.00 -> 56.3 mm
- net Net-(T1-OUT2A): track 26.4 -> 0.00 mm
- net Net-(T1-OUT2B): track 26.2 -> 0.00 mm
- net 18VAC-: track 61.8 -> 38.6 mm
- net INV_OUTB: track 56.1 -> 35.5 mm
- net SHUNT: track 250.4 -> 266.3 mm
- net 12V: track 158.0 -> 170.9 mm
- net +BATT: track 70.6 -> 83.4 mm
- net 380V: track 214.9 -> 221.8 mm, vias 0 -> 1
- net Net-(J6-Pin_1): track 56.8 -> 51.4 mm
- net INV_OUTA: track 46.0 -> 41.6 mm
- net Net-(J6-Pin_2): track 71.6 -> 67.8 mm
- net -BATT: track 158.1 -> 161.7 mm
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- added copper zone on F.Cu, net -BATT
- added copper zone on F.Cu, net INV_TR+
- added copper zone on F.Cu, net INV_TR-
Other:
- outline, holes or cut-outs redrawn
- board text added: "18VAC 18V 12V 5V"
- board text added: "AC"
- board text added: "AC EN"
- board text added: "DC"
- board text added: "DC EN"
- board text added: "I2C"
- board text added: "PRG"
- board text added: "RST"
- board text added: "SPI"
- board text added: "STATUS"
- board text added: "UART"
