File: VoltPak-1000/VolPak-1000/VolPak-1000.kicad_sch (KiCad schematic)
At the start: 185 parts, among them J1 USB_C_Receptacle_USB2.0_14P, J10 UART JST, J11 USB_A, J12 USB_C_Receptacle_USB2.0_14P, J2 SPI JST, J3 Input Switch, J4 12V Battery Input, J5 Fan Connector, J6 AC Outlet, J7 EGS002, J8 I2C JST, J9 POWER JST, Q1 SS8050, Q10 FGH40N65, Q11 FGH40N65, Q12 S8050, Q13 S8050, Q2 SS8050, Q3 IRF3205, Q4 IRF3205, Q5 IRF3205, Q6 IRF3205, Q7 SS8050, Q8 FGH40N65, Q9 FGH40N65, SW1 SW_Push, SW2 SW_Push, SW4 SW_Push, SW5 SW_Push, T1 E55, U1 ESP32-S3, U10 AP63203WU, U11 AP63205WU, U2 W25Q128JVS, U3 CP2102N-Axx-xQFN28, U4 LD1117S18TR_SOT223, U5 SG3525, U6 L7812, U7 L7805, U8 INA219BxDCN, U9 INA219BxDCN, Y1 40MHz (+/-10PPM)

Commit message: more circuit stuff
Parts:
- C28, C32: footprint (none) -> Capacitor_THT:CP_Radial_D10.0mm_P5.00mm; LCSC (none) -> C503217
- C30: footprint (none) -> Capacitor_THT:CP_Radial_D5.0mm_P2.00mm; LCSC (none) -> C2960204
- C31, C34, C50, C52: value 100nF -> 0.1uF
- C33, C37: footprint (none) -> Capacitor_THT:CP_Radial_D8.0mm_P3.80mm; LCSC (none) -> C7499907
- C35, C36: footprint (none) -> Capacitor_THT:CP_Radial_D18.0mm_P7.50mm; LCSC (none) -> C2843909
- C38, C39: footprint (none) -> Capacitor_THT:CP_Radial_D16.0mm_P7.50mm; LCSC (none) -> C711636
- C40: value 100nF 275VAC -> 0.1uF 275VAC; footprint (none) -> Capacitor_THT:C_Disc_D4.3mm_W1.9mm_P5.00mm; LCSC (none) -> C600230
- C41, C42: value 100nF -> 0.1uF; footprint (none) -> Capacitor_SMD:C_0603_1608Metric
- C43: footprint (none) -> Capacitor_SMD:C_0603_1608Metric
- C7, C8: footprint (none) -> Capacitor_SMD:C_0402_1005Metric
- D10, D11, D12, D13, D14, D15, D16, D17: footprint (none) -> Diode_THT:D_DO-15_P3.81mm_Vertical_KathodeUp
- D6, D7, D9: footprint (none) -> LED_SMD:LED_0603_1608Metric; LCSC (none) -> C7501578
- J10, J8: footprint (none) -> Connector_JST:JST_EH_B2B-EH-A_1x02_P2.50mm_Vertical
- J2: footprint (none) -> Connector_JST:JST_EH_B6B-EH-A_1x06_P2.50mm_Vertical
- J4, J6: footprint (none) -> TerminalBlock:TerminalBlock_MaiXu_MX126-5.0-02P_1x02_P5.00mm; LCSC (none) -> C8269
- J5: footprint (none) -> Connector_PinHeader_2.54mm:PinHeader_1x02_P2.54mm_Vertical
- J9: footprint (none) -> Connector_JST:JST_EH_B4B-EH-A_1x04_P2.50mm_Vertical
- L1, L2, L4, L5: footprint (none) -> Inductor_SMD:L_0402_1005Metric
- L3: value L -> 2.5MH 10.0A
- R1, R10, R11, R12, R13, R14, R15, R16, R17, R18, R19, R2, R20, R21, R22, R24, R25, R26, R3, R4, R43, R5, R54, R55, R56, R57, R58, R59, R6, R60, R61, R64, R65, R7, R8, R9: footprint (none) -> Resistor_SMD:R_0402_1005Metric
- R23, R27, R28, R29, R30, R31, R32, R33, R34, R35, R36, R37, R40, R41, R42, R44, R45, R46, R47, R48, R49, R50, R51, R52, R53: footprint (none) -> Resistor_SMD:R_0603_1608Metric
- R38, R39: footprint (none) -> Resistor_SMD:R_0815_2038Metric
- RV1: footprint (none) -> Potentiometer_THT:Potentiometer_Bourns_3296W_Vertical; LCSC (none) -> C118954

Commit message: finished layout, yet to source parts
Parts:
- removed Q10, Q8, Q9: FGH40N65, symbol Device:Q_NIGBT_CGE
- added Q10, Q8, Q9: FGH40N65, symbol Device:Q_NIGBT_GCE
- added R62: 0, Resistor_SMD:R_0402_1005Metric, symbol Device:R
- C7, C8: value TBD -> 6pF
- CHOKE1: renamed from TR1; value TRANSF1 -> 2.5MH 10A; footprint (none) -> Inductor_THT:Choke_Schaffner_RN216-04-15.5x23.0mm
- J1: footprint (none) -> Connector_USB:USB_C_Receptacle_G-Switch_GT-USB-7010ASV; LCSC (none) -> C2765186
- J11: footprint (none) -> Connector_USB:USB_A_Molex_67643_Horizontal; LCSC (none) -> C591765
- J12: footprint (none) -> Connector_USB:USB_C_C783299; LCSC (none) -> C783299
- J3: footprint (none) -> Connector_PinHeader_2.54mm:PinHeader_1x03_P2.54mm_Vertical
- J7: footprint (none) -> Connector_PinHeader_2.54mm:PinHeader_1x17_P2.54mm_Vertical
- L3: value 2.5MH 10.0A -> 2.5MH 10A; footprint (none) -> Inductor_THT:L_Toroid_Vertical_L48.8mm_W25.4mm_P20.80mm_Vishay_TJ8; LCSC (none) -> C2831473
- Q11: symbol Device:Q_NIGBT_CGE -> Device:Q_NIGBT_GCE
- R20: value 0 -> 0R
- R8: value 0 -> 24nH; footprint Resistor_SMD:R_0402_1005Metric -> Inductor_SMD:L_0402_1005Metric; symbol Device:R -> Device:L
- T1: footprint (none) -> Transformer_THT:Transformer_CHK_EI54-12VA_Neutral
- U5: footprint (none) -> Package_SO:SOP-16_3.9x9.9mm_P1.27mm; LCSC (none) -> C7598682
- U6: footprint (none) -> Package_TO_SOT_THT:TO-220-3_Vertical; LCSC (none) -> C2914
- U7: footprint (none) -> Package_TO_SOT_THT:TO-220-3_Vertical; LCSC (none) -> C3795
- Y1: value 40MHz (+/-10PPM) -> 40MHz +/-10PPM 8pF; footprint (none) -> Crystal:Crystal_SMD_3225-4Pin_3.2x2.5mm; LCSC (none) -> C7294596
Connections:
- net 380V: now also Q8.2 (C), Q9.2 (C)
- net 5V: now also R62.1; no longer R53.2, U9.2 (IN-)
- net CHIP_PU: now also R20.1; no longer R20.2
- net CH_L: now also Q10.2 (C), Q9.3 (E)
- net COIL: now also Q11.2 (C), Q8.3 (E); no longer Q11.1 (C)
- net GPIO0: now also R21.1; no longer R21.2
- net SHUNT: now also Q10.3 (E)
- net at R44.2: now also Q9.1 (G)
- net at R49.2: now also Q11.1 (G); no longer Q11.2 (G)
- net at R46.2: now also Q10.1 (G)
- net at Q2.3 (C): now also R20.2; no longer R20.1
- net at Q1.3 (C): now also R21.2; no longer R21.1
- net at R48.2: now also Q8.1 (G)
- new net: R53.2, R62.2, U9.2 (IN-)
Other:
- moved on the sheet: C27, C44, R20, R21, R23, R54, R55, U8

Commit message: completed layout
Parts:
- A1, J10, J2, J3, J5, J7, J8, J9, T1: LCSC (none) -> -
- C1, C13, C14, C17, C18, C2, C20, C21, C23, C26, C27, C31, C34, C4, C46, C50, C52: LCSC (none) -> C6119799
- C10, C9: LCSC (none) -> C880658
- C11, C15, C22, C24, C25, C44, C45, C47, C51: LCSC (none) -> C23692971
- C12, C16, C19, C3, C6: LCSC (none) -> C2887021
- C29, C5: LCSC (none) -> C688874
- C40: footprint Capacitor_THT:C_Disc_D4.3mm_W1.9mm_P5.00mm -> Capacitor_SMD:C_2220_5750Metric_Pad1.97x5.40mm_HandSolder; LCSC C600230 -> C5290327
- C41, C42: footprint Capacitor_SMD:C_0603_1608Metric -> Capacitor_SMD:C_2220_5750Metric_Pad1.97x5.40mm_HandSolder; LCSC (none) -> C5290327
- C43: LCSC (none) -> C100042
- C48, C49, C53, C54: LCSC (none) -> C415703
- C7, C8: LCSC (none) -> C437443
- CHOKE1: value 2.5MH 10A -> 2MH 10A; LCSC (none) -> C2831473
- D1, D3, D4: LCSC (none) -> C5180230
- D10, D11, D12, D13: LCSC (none) -> C31251
- D14, D15, D16, D17: LCSC (none) -> C402212
- D18: LCSC (none) -> C5632681
- D2: LCSC (none) -> C5380881
- D5: LCSC (none) -> C110032
- L1: LCSC (none) -> C76769
- L2: LCSC (none) -> C913678
- L3: LCSC C2831473 -> -
- L4: LCSC (none) -> C18221128
- L5: footprint Inductor_SMD:L_0402_1005Metric -> Inductor_SMD:L_0603_1608Metric; LCSC (none) -> C22447690
- Q1, Q2, Q7: LCSC (none) -> C2834467
- Q10, Q11, Q8, Q9: footprint (none) -> Package_TO_SOT_THT:TO-247-3_Vertical; LCSC (none) -> C472600
- Q12, Q13: LCSC (none) -> C2931492
- Q3, Q4, Q5, Q6: LCSC (none) -> C19189952
- R1, R10, R15, R16, R17, R2, R20, R21, R22, R3, R4, R5, R62: LCSC (none) -> C106231
- R11: LCSC (none) -> C25896
- R12: LCSC (none) -> C163478
- R13, R54, R55: LCSC (none) -> C11702
- R14, R18, R19, R56, R57, R64, R65, R7, R9: LCSC (none) -> C60490
- R23, R53: LCSC (none) -> https://www.digikey.ca/en/products/detail/panasonic-electro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
- R24: LCSC (none) -> C137992
- R25, R26, R58, R60: LCSC (none) -> C25905
- R27, R28, R29, R30, R33, R35, R37: LCSC (none) -> C161787
- R31: LCSC (none) -> C2907028
- R32, R44, R46, R48, R49: LCSC (none) -> C109318
- R34, R36: LCSC (none) -> C2907045
- R38, R39: footprint Resistor_SMD:R_0815_2038Metric -> Resistor_SMD:R_2512_6332Metric; LCSC (none) -> C469426
- R40, R45, R47, R50, R51: LCSC (none) -> C2907046
- R41, R42: LCSC (none) -> C491207
- R43: LCSC (none) -> C4109
- R52: LCSC (none) -> C137705
- R59, R61: LCSC (none) -> C2909336
- R6: LCSC (none) -> C137970
- R8: LCSC (none) -> C404641
- SW1, SW2, SW4, SW5: LCSC (none) -> C221895
- TH1: LCSC (none) -> C394024
- U1: LCSC (none) -> https://www.digikey.ca/en/products/detail/espressif-systems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
- U10: LCSC (none) -> C780769
- U11: LCSC (none) -> C2071056
- U2: LCSC (none) -> C113767
- U3: LCSC (none) -> C964632
- U4: LCSC (none) -> C19627011
- U8, U9: LCSC (none) -> C962069
Connections:
- net +BATT: now also T1.5 (VCC), T1.6 (VCC), T1.7 (VCC); no longer T1.2 (PM)
- net 18VAC+: now also T1.12 (OUT-); no longer T1.4 (OUT1A)
- net 18VAC-: now also T1.13 (NC13); no longer T1.5 (OUT1B)
- net INV_TR+: now also T1.2 (IN-), T1.3 (IN-)
- net INV_TR-: now also T1.10 (IN+), T1.11 (IN+), T1.9 (IN+); no longer T1.3 (IN-)
- net at D18.3: now also T1.16 (NC16); no longer T1.6 (OUT2A)
- net at D18.2: now also T1.22 (AUX+); no longer T1.7 (OUT2B)
- no-connect marks 27 -> 36
Other:
- note added: "KW Inverter"
- note removed: "0.5KW Inverter"

Commit message: generated plots
Other:
- note added: "1000W Pure Sine Wave Inverter"
- note added: "Auto program table"
- note added: "USB Power Ports"
- note removed: "Auto program DTR RTS-->EN IO0 IO2 1 1 1 1 1 0 0 1 1 1 1 0 0 1 1 0 1 1 0 0"
- note removed: "KW Inverter"
- company: (none) -> VoltPak © Diskovery Group Limited
- title: (none) -> VoltPak-1000 Version 0.1
- moved on the sheet: A1, C1, C10, C11, C12, C13, C14, C15, C16, C17, C18, C19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
